Commit message: expand urdf to have prototype full leg

File: urdf/model.urdf.xacro (robot description, xacro)
@@ -1,10 +1,93 @@
 <?xml version="1.0"?>
-<robot name="myfirst">
+<robot name="ALEX_Model" xmlns:xacro="http://www.ros.org/wiki/xacro">
   <link name="base_link">
     <visual>
       <geometry>
-        <cylinder length="0.6" radius="0.2"/>
+        <box size="0.5 0.01 0.2" />
       </geometry>
+      <origin xyz="0 0 1"/>
     </visual>
   </link>
+  <link name="right_hip">
+    <visual>
+      <geometry>
+        <cylinder length="0.2" radius="0.02" />
+      </geometry>
+      <origin xyz="0.1 0 0" rpy="0 ${pi / 2} 0"/>
+    </visual>
+  </link>
+  <joint name="base_to_right_hip" type="fixed">
+    <parent link="base_link"/>
+    <child link="right_hip"/>
+    <origin xyz="0.25 0 1"/>
+  </joint>
+  <link name="right_thigh">
+    <visual>
+      <geometry>
+        <cylinder length="0.4" radius="0.1" />
+      </geometry>
+      <origin xyz="0 0 -0.2" />
+    </visual>
+  </link>
+  <joint name="right_hip_to_thigh" type="revolute">
+    <parent link="right_hip" />
+    <child link="right_thigh" />
+    <origin xyz="0.1 0 0" />
+    <axis xyz="1 0 0" rpy="0 0 0"/>
+    <limit lower="${-pi / 2}" upper="${pi / 2}" effort="100" velocity="1" />
+  </joint>
+  <link name="right_knee">
+    <visual>
+      <geometry>
+        <cylinder length="0.15" radius="0.02" />
+      </geometry>
+      <origin xyz="0 0 0" rpy="0 ${pi / 2} 0"/>
+    </visual>
+  </link>
+  <joint name="right_thigh_to_knee" type="fixed">
+    <parent link="right_thigh" />
+    <child link="right_knee" />
+    <origin xyz="0 0 -0.4" />
+  </joint>
+  <link name="right_calf">
+    <visual>
+      <geometry>
+        <cylinder length="0.3" radius="0.075" />
+      </geometry>
+      <origin xyz="0 0 -0.15" rpy="0 0 0" />
+    </visual>
+  </link>
+  <joint name="right_knee_to_calf" type="revolute">
+    <parent link="right_knee" />
+    <child link="right_calf" />
+    <origin xyz="0 0 0" />
+    <axis xyz="1 0 0" rpy="0 0 0"/>
+    <limit lower="${-pi / 2}" upper="${pi / 2}" effort="100" velocity="1" />
+  </joint>
+  <link name="right_ankle">
+    <visual>
+      <geometry>
+        <cylinder length="0.1" radius="0.02" />
+      </geometry>
+      <origin xyz="0 0 0" rpy="0 ${pi / 2} 0"/>
+    </visual>
+  </link>
+  <joint name="right_calf_to_ankle" type="fixed">
+    <parent link="right_calf" />
+    <child link="right_ankle" />
+    <origin xyz="0 0 -0.3" />
+  </joint>
+  <link name="right_foot">
+    <visual>
+      <geometry>
+        <box size="0.1 0.2 0.01"/>
+      </geometry>
+      <origin xyz="0 -0.05 0"/>
+    </visual>
+  </link>
+  <joint name="right_ankle_to_foot" type="fixed">
+    <parent link="right_ankle" />
+    <child link="right_foot" />
+    <origin xyz="0 0 -0.02" />
+  </joint>
 </robot>

Commit message: now launching with gazebo

File: urdf/model.urdf.xacro (robot description, xacro)
@@ -1,4 +1,5 @@
 <?xml version="1.0"?>
 <robot name="ALEX_Model" xmlns:xacro="http://www.ros.org/wiki/xacro">
+  <link name="world"></link>
   <link name="base_link">
     <visual>
@@ -6,7 +7,23 @@
         <box size="0.5 0.01 0.2" />
       </geometry>
-      <origin xyz="0 0 1"/>
+      <origin xyz="0 0 0" />
     </visual>
+    <collision>
+      <geometry>
+        <box size="0.5 0.01 0.2" />
+      </geometry>
+      <origin xyz="0 0 0" />
+    </collision>
+    <inertial>
+      <origin xyz="0 0 0" rpy="0 0 0"/>
+      <mass value="12" />
+      <inertia ixx="2.26" ixy="0.0" ixz="0.0" iyy="6.26" iyz="0.0" izz="8.5" />
+    </inertial>
   </link>
+  <joint name="base_joint" type="fixed">
+    <parent link="world"/>
+    <child link="base_link"/>
+    <origin xyz="0 0 1" rpy="0 0 0"/>
+  </joint>
   <link name="right_hip">
     <visual>
@@ -16,9 +33,20 @@
       <origin xyz="0.1 0 0" rpy="0 ${pi / 2} 0"/>
     </visual>
+    <collision>
+      <geometry>
+        <cylinder length="0.2" radius="0.02" />
+      </geometry>
+      <origin xyz="0.1 0 0" rpy="0 ${pi / 2} 0"/>
+    </collision>
+    <inertial>
+      <origin xyz="0 0 0" rpy="0 0 0"/>
+      <mass value="12" />
+      <inertia ixx="2.26" ixy="0.0" ixz="0.0" iyy="6.26" iyz="0.0" izz="8.5" />
+    </inertial>
   </link>
   <joint name="base_to_right_hip" type="fixed">
     <parent link="base_link"/>
     <child link="right_hip"/>
-    <origin xyz="0.25 0 1"/>
+    <origin xyz="0.25 0 0"/>
   </joint>
   <link name="right_thigh">
@@ -29,4 +57,15 @@
       <origin xyz="0 0 -0.2" />
     </visual>
+    <collision>
+      <geometry>
+        <cylinder length="0.4" radius="0.1" />
+      </geometry>
+      <origin xyz="0 0 -0.2" />
+    </collision>
+    <inertial>
+      <origin xyz="0 0 0" rpy="0 0 0"/>
+      <mass value="12" />
+      <inertia ixx="2.26" ixy="0.0" ixz="0.0" iyy="6.26" iyz="0.0" izz="8.5" />
+    </inertial>
   </link>
   <joint name="right_hip_to_thigh" type="revolute">
@@ -44,4 +83,15 @@
       <origin xyz="0 0 0" rpy="0 ${pi / 2} 0"/>
     </visual>
+    <collision>
+      <geometry>
+        <cylinder length="0.15" radius="0.02" />
+      </geometry>
+      <origin xyz="0 0 0" rpy="0 ${pi / 2} 0"/>
+    </collision>
+    <inertial>
+      <origin xyz="0 0 0" rpy="0 0 0"/>
+      <mass value="12" />
+      <inertia ixx="2.26" ixy="0.0" ixz="0.0" iyy="6.26" iyz="0.0" izz="8.5" />
+    </inertial>
   </link>
   <joint name="right_thigh_to_knee" type="fixed">
@@ -57,4 +107,15 @@
       <origin xyz="0 0 -0.15" rpy="0 0 0" />
     </visual>
+    <collision>
+      <geometry>
+        <cylinder length="0.3" radius="0.075" />
+      </geometry>
+      <origin xyz="0 0 -0.15" rpy="0 0 0" />
+    </collision>
+    <inertial>
+      <origin xyz="0 0 0" rpy="0 0 0"/>
+      <mass value="12" />
+      <inertia ixx="2.26" ixy="0.0" ixz="0.0" iyy="6.26" iyz="0.0" izz="8.5" />
+    </inertial>
   </link>
   <joint name="right_knee_to_calf" type="revolute">
@@ -72,4 +133,15 @@
       <origin xyz="0 0 0" rpy="0 ${pi / 2} 0"/>
     </visual>
+    <collision>
+      <geometry>
+        <cylinder length="0.1" radius="0.02" />
+      </geometry>
+      <origin xyz="0 0 0" rpy="0 ${pi / 2} 0"/>
+    </collision>
+    <inertial>
+      <origin xyz="0 0 0" rpy="0 0 0"/>
+      <mass value="12" />
+      <inertia ixx="2.26" ixy="0.0" ixz="0.0" iyy="6.26" iyz="0.0" izz="8.5" />
+    </inertial>
   </link>
   <joint name="right_calf_to_ankle" type="fixed">
@@ -85,4 +157,15 @@
       <origin xyz="0 -0.05 0"/>
     </visual>
+    <collision>
+      <geometry>
+        <box size="0.1 0.2 0.01"/>
+      </geometry>
+      <origin xyz="0 -0.05 0"/>
+    </collision>
+    <inertial>
+      <origin xyz="0 0 0" rpy="0 0 0"/>
+      <mass value="12" />
+      <inertia ixx="2.26" ixy="0.0" ixz="0.0" iyy="6.26" iyz="0.0" izz="8.5" />
+    </inertial>
   </link>
   <joint name="right_ankle_to_foot" type="fixed">

Commit message: clean up xacro with macros

File: urdf/model.urdf.xacro (robot description, xacro)
@@ -1,71 +1,27 @@
 <?xml version="1.0"?>
 <robot name="ALEX_Model" xmlns:xacro="http://www.ros.org/wiki/xacro">
+  <xacro:include filename="common.xacro" />
   <link name="world"></link>
-  <link name="base_link">
-    <visual>
-      <geometry>
-        <box size="0.5 0.01 0.2" />
-      </geometry>
-      <origin xyz="0 0 0" />
-    </visual>
-    <collision>
-      <geometry>
-        <box size="0.5 0.01 0.2" />
-      </geometry>
-      <origin xyz="0 0 0" />
-    </collision>
-    <inertial>
-      <origin xyz="0 0 0" rpy="0 0 0"/>
-      <mass value="12" />
-      <inertia ixx="2.26" ixy="0.0" ixz="0.0" iyy="6.26" iyz="0.0" izz="8.5" />
-    </inertial>
+  <link name="back_plate">
+    <xacro:box_visual_and_collision size="0.5 0.01 0.2" xyz="0 0 0"/>
+    <xacro:generic_inertia />
   </link>
   <joint name="base_joint" type="fixed">
     <parent link="world"/>
-    <child link="base_link"/>
+    <child link="back_plate"/>
     <origin xyz="0 0 1" rpy="0 0 0"/>
   </joint>
   <link name="right_hip">
-    <visual>
-      <geometry>
-        <cylinder length="0.2" radius="0.02" />
-      </geometry>
-      <origin xyz="0.1 0 0" rpy="0 ${pi / 2} 0"/>
-    </visual>
-    <collision>
-      <geometry>
-        <cylinder length="0.2" radius="0.02" />
-      </geometry>
-      <origin xyz="0.1 0 0" rpy="0 ${pi / 2} 0"/>
-    </collision>
-    <inertial>
-      <origin xyz="0 0 0" rpy="0 0 0"/>
-      <mass value="12" />
-      <inertia ixx="2.26" ixy="0.0" ixz="0.0" iyy="6.26" iyz="0.0" izz="8.5" />
-    </inertial>
+    <xacro:cylinder_visual_and_collision length="0.2" radius="0.02" xyz="0.1 0 0" rpy="0 ${pi/2} 0" />
+    <xacro:generic_inertia />
   </link>
   <joint name="base_to_right_hip" type="fixed">
-    <parent link="base_link"/>
+    <parent link="back_plate"/>
     <child link="right_hip"/>
     <origin xyz="0.25 0 0"/>
   </joint>
   <link name="right_thigh">
-    <visual>
-      <geometry>
-        <cylinder length="0.4" radius="0.1" />
-      </geometry>
-      <origin xyz="0 0 -0.2" />
-    </visual>
-    <collision>
-      <geometry>
-        <cylinder length="0.4" radius="0.1" />
-      </geometry>
-      <origin xyz="0 0 -0.2" />
-    </collision>
-    <inertial>
-      <origin xyz="0 0 0" rpy="0 0 0"/>
-      <mass value="12" />
-      <inertia ixx="2.26" ixy="0.0" ixz="0.0" iyy="6.26" iyz="0.0" izz="8.5" />
-    </inertial>
+    <xacro:cylinder_visual_and_collision length="0.4" radius="0.1" xyz="0 0 -0.2" rpy="0 0 0" />
+    <xacro:generic_inertia />
   </link>
   <joint name="right_hip_to_thigh" type="revolute">
@@ -77,21 +33,6 @@
   </joint>
   <link name="right_knee">
-    <visual>
-      <geometry>
-        <cylinder length="0.15" radius="0.02" />
-      </geometry>
-      <origin xyz="0 0 0" rpy="0 ${pi / 2} 0"/>
-    </visual>
-    <collision>
-      <geometry>
-        <cylinder length="0.15" radius="0.02" />
-      </geometry>
-      <origin xyz="0 0 0" rpy="0 ${pi / 2} 0"/>
-    </collision>
-    <inertial>
-      <origin xyz="0 0 0" rpy="0 0 0"/>
-      <mass value="12" />
-      <inertia ixx="2.26" ixy="0.0" ixz="0.0" iyy="6.26" iyz="0.0" izz="8.5" />
-    </inertial>
+    <xacro:cylinder_visual_and_collision length="0.15" radius="0.02" xyz="0 0 0" rpy="0 ${pi / 2} 0" />
+    <xacro:generic_inertia />
   </link>
   <joint name="right_thigh_to_knee" type="fixed">
@@ -101,21 +42,6 @@
   </joint>
   <link name="right_calf">
-    <visual>
-      <geometry>
-        <cylinder length="0.3" radius="0.075" />
-      </geometry>
-      <origin xyz="0 0 -0.15" rpy="0 0 0" />
-    </visual>
-    <collision>
-      <geometry>
-        <cylinder length="0.3" radius="0.075" />
-      </geometry>
-      <origin xyz="0 0 -0.15" rpy="0 0 0" />
-    </collision>
-    <inertial>
-      <origin xyz="0 0 0" rpy="0 0 0"/>
-      <mass value="12" />
-      <inertia ixx="2.26" ixy="0.0" ixz="0.0" iyy="6.26" iyz="0.0" izz="8.5" />
-    </inertial>
+    <xacro:cylinder_visual_and_collision length="0.3" radius="0.075" xyz="0 0 -0.15" rpy="0 0 0" />
+    <xacro:generic_inertia />
   </link>
   <joint name="right_knee_to_calf" type="revolute">
@@ -127,21 +53,6 @@
   </joint>
   <link name="right_ankle">
-    <visual>
-      <geometry>
-        <cylinder length="0.1" radius="0.02" />
-      </geometry>
-      <origin xyz="0 0 0" rpy="0 ${pi / 2} 0"/>
-    </visual>
-    <collision>
-      <geometry>
-        <cylinder length="0.1" radius="0.02" />
-      </geometry>
-      <origin xyz="0 0 0" rpy="0 ${pi / 2} 0"/>
-    </collision>
-    <inertial>
-      <origin xyz="0 0 0" rpy="0 0 0"/>
-      <mass value="12" />
-      <inertia ixx="2.26" ixy="0.0" ixz="0.0" iyy="6.26" iyz="0.0" izz="8.5" />
-    </inertial>
+    <xacro:cylinder_visual_and_collision length="0.1" radius="0.02" xyz="0 0 0" rpy="0 ${pi / 2} 0" />
+    <xacro:generic_inertia />
   </link>
   <joint name="right_calf_to_ankle" type="fixed">
@@ -151,21 +62,6 @@
   </joint>
   <link name="right_foot">
-    <visual>
-      <geometry>
-        <box size="0.1 0.2 0.01"/>
-      </geometry>
-      <origin xyz="0 -0.05 0"/>
-    </visual>
-    <collision>
-      <geometry>
-        <box size="0.1 0.2 0.01"/>
-      </geometry>
-      <origin xyz="0 -0.05 0"/>
-    </collision>
-    <inertial>
-      <origin xyz="0 0 0" rpy="0 0 0"/>
-      <mass value="12" />
-      <inertia ixx="2.26" ixy="0.0" ixz="0.0" iyy="6.26" iyz="0.0" izz="8.5" />
-    </inertial>
+    <xacro:box_visual_and_collision size="0.1 0.2 0.01" xyz="0 -0.05 0"/>
+    <xacro:generic_inertia />
   </link>
   <joint name="right_ankle_to_foot" type="fixed">

Commit message: add property variables

File: urdf/model.urdf.xacro (robot description, xacro)
@@ -3,6 +3,7 @@
   <xacro:include filename="common.xacro" />
   <link name="world"></link>
+  <xacro:property name="back_plate_width" value="0.5" />
   <link name="back_plate">
-    <xacro:box_visual_and_collision size="0.5 0.01 0.2" xyz="0 0 0"/>
+    <xacro:box_visual_and_collision size="${back_plate_width} 0.01 0.2" xyz="0 0 0"/>
     <xacro:generic_inertia />
   </link>
@@ -12,6 +13,8 @@
     <origin xyz="0 0 1" rpy="0 0 0"/>
   </joint>
+<!--
+  <xacro:property name="hip_width" value="0.2" />
   <link name="right_hip">
-    <xacro:cylinder_visual_and_collision length="0.2" radius="0.02" xyz="0.1 0 0" rpy="0 ${pi/2} 0" />
+    <xacro:cylinder_visual_and_collision length="${hip_width}" radius="0.02" xyz="0.1 0 0" rpy="0 ${pi/2} 0" />
     <xacro:generic_inertia />
   </link>
@@ -19,8 +22,9 @@
     <parent link="back_plate"/>
     <child link="right_hip"/>
-    <origin xyz="0.25 0 0"/>
+    <origin xyz="${back_plate_width / 2} 0 0"/>
   </joint>
+  <xacro:property name="thigh_length" value="0.4" />
   <link name="right_thigh">
-    <xacro:cylinder_visual_and_collision length="0.4" radius="0.1" xyz="0 0 -0.2" rpy="0 0 0" />
+    <xacro:cylinder_visual_and_collision length="${thigh_length}" radius="0.1" xyz="0 0 -0.2" rpy="0 0 0" />
     <xacro:generic_inertia />
   </link>
@@ -28,10 +32,11 @@
     <parent link="right_hip" />
     <child link="right_thigh" />
-    <origin xyz="0.1 0 0" />
+    <origin xyz="${hip_width / 2} 0 0" />
     <axis xyz="1 0 0" rpy="0 0 0"/>
     <limit lower="${-pi / 2}" upper="${pi / 2}" effort="100" velocity="1" />
   </joint>
+  <xacro:property name="knee_width" value="0.15" />
   <link name="right_knee">
-    <xacro:cylinder_visual_and_collision length="0.15" radius="0.02" xyz="0 0 0" rpy="0 ${pi / 2} 0" />
+    <xacro:cylinder_visual_and_collision length="${knee_width}" radius="0.02" xyz="0 0 0" rpy="0 ${pi / 2} 0" />
     <xacro:generic_inertia />
   </link>
@@ -39,8 +44,9 @@
     <parent link="right_thigh" />
     <child link="right_knee" />
-    <origin xyz="0 0 -0.4" />
+    <origin xyz="0 0 ${-1 * thigh_length}" />
   </joint>
+  <xacro:property name="calf_length" value="0.3" />
   <link name="right_calf">
-    <xacro:cylinder_visual_and_collision length="0.3" radius="0.075" xyz="0 0 -0.15" rpy="0 0 0" />
+    <xacro:cylinder_visual_and_collision length="${calf_length}" radius="0.075" xyz="0 0 -0.15" rpy="0 0 0" />
     <xacro:generic_inertia />
   </link>
@@ -52,6 +58,7 @@
     <limit lower="${-pi / 2}" upper="${pi / 2}" effort="100" velocity="1" />
   </joint>
+  <xacro:property name="ankle_radius" value="0.02" />
   <link name="right_ankle">
-    <xacro:cylinder_visual_and_collision length="0.1" radius="0.02" xyz="0 0 0" rpy="0 ${pi / 2} 0" />
+    <xacro:cylinder_visual_and_collision length="0.1" radius="${ankle_radius}" xyz="0 0 0" rpy="0 ${pi / 2} 0" />
     <xacro:generic_inertia />
   </link>
@@ -59,5 +66,5 @@
     <parent link="right_calf" />
     <child link="right_ankle" />
-    <origin xyz="0 0 -0.3" />
+    <origin xyz="0 0 ${-1 * calf_length}" />
   </joint>
   <link name="right_foot">
@@ -68,5 +75,5 @@
     <parent link="right_ankle" />
     <child link="right_foot" />
-    <origin xyz="0 0 -0.02" />
-  </joint>
+    <origin xyz="0 0 ${-1 * ankle_radius}" />
+  </joint> -->
 </robot>

Commit message: Update model.urdf.xacro

File: urdf/model.urdf.xacro (robot description, xacro)
@@ -13,5 +13,4 @@
     <origin xyz="0 0 1" rpy="0 0 0"/>
   </joint>
-<!--
   <xacro:property name="hip_width" value="0.2" />
   <link name="right_hip">
@@ -76,4 +75,4 @@
     <child link="right_foot" />
     <origin xyz="0 0 ${-1 * ankle_radius}" />
-  </joint> -->
+  </joint>
 </robot>

Commit message: camera works

File: urdf/model.urdf.xacro (robot description, xacro)
@@ -2,4 +2,7 @@
 <robot name="ALEX_Model" xmlns:xacro="http://www.ros.org/wiki/xacro">
   <xacro:include filename="common.xacro" />
+  <gazebo reference="back_plate">
+    <material>Gazebo/Orange</material>
+  </gazebo>
   <link name="world"></link>
   <xacro:property name="back_plate_width" value="0.5" />
@@ -76,3 +79,53 @@
     <origin xyz="0 0 ${-1 * ankle_radius}" />
   </joint>
+  <gazebo>
+    <plugin name="gazebo_ros_joint_state_publisher"
+        filename="libgazebo_ros_joint_state_publisher.so">
+        <update_rate>20</update_rate>
+        <joint_name>base_to_right_hip</joint_name>
+        <joint_name>right_hip_to_thigh</joint_name>
+        <joint_name>right_thigh_to_knee</joint_name>
+        <joint_name>right_knee_to_calf</joint_name>
+        <joint_name>right_calf_to_ankle</joint_name>
+    </plugin>
+  </gazebo>
+  <gazebo reference="right_foot">
+    <sensor type="camera" name="camera1">
+      <update_rate>30.0</update_rate>
+      <camera name="head">
+        <horizontal_fov>1.3962634</horizontal_fov>
+        <image>
+          <width>800</width>
+          <height>800</height>
+          <format>R8G8B8</format>
+        </image>
+        <clip>
+          <near>0.02</near>
+          <far>300</far>
+        </clip>
+        <noise>
+          <type>gaussian</type>
+          <!-- Noise is sampled independently per pixel on each frame.
+               That pixel's noise value is added to each of its color
+               channels, which at that point lie in the range [0,1]. -->
+          <mean>0.0</mean>
+          <stddev>0.007</stddev>
+        </noise>
+      </camera>
+      <plugin name="camera_controller" filename="libgazebo_ros_camera.so">
+        <alwaysOn>true</alwaysOn>
+        <updateRate>0.0</updateRate>
+        <cameraName>ALEX_Model/camera1</cameraName>
+        <imageTopicName>image_raw</imageTopicName>
+        <cameraInfoTopicName>camera_info</cameraInfoTopicName>
+        <frameName>right_foot</frameName>
+        <hackBaseline>0.07</hackBaseline>
+        <distortionK1>0.0</distortionK1>
+        <distortionK2>0.0</distortionK2>
+        <distortionK3>0.0</distortionK3>
+        <distortionT1>0.0</distortionT1>
+        <distortionT2>0.0</distortionT2>
+      </plugin>
+    </sensor>
+  </gazebo>
 </robot>

Commit message: add imu sensor

File: urdf/model.urdf.xacro (robot description, xacro)
@@ -21,4 +21,7 @@
     <xacro:generic_inertia />
   </link>
+  <gazebo reference="right_hip">
+    <material>Gazebo/Blue</material>
+  </gazebo>
   <joint name="base_to_right_hip" type="fixed">
     <parent link="back_plate"/>
@@ -31,4 +34,7 @@
     <xacro:generic_inertia />
   </link>
+  <gazebo reference="right_thigh">
+    <material>Gazebo/Blue</material>
+  </gazebo>
   <joint name="right_hip_to_thigh" type="revolute">
     <parent link="right_hip" />
@@ -43,4 +49,7 @@
     <xacro:generic_inertia />
   </link>
+  <gazebo reference="right_knee">
+    <material>Gazebo/Blue</material>
+  </gazebo>
   <joint name="right_thigh_to_knee" type="fixed">
     <parent link="right_thigh" />
@@ -53,4 +62,7 @@
     <xacro:generic_inertia />
   </link>
+  <gazebo reference="right_calf">
+    <material>Gazebo/Blue</material>
+  </gazebo>
   <joint name="right_knee_to_calf" type="revolute">
     <parent link="right_knee" />
@@ -65,4 +77,7 @@
     <xacro:generic_inertia />
   </link>
+  <gazebo reference="right_ankle">
+    <material>Gazebo/Blue</material>
+  </gazebo>
   <joint name="right_calf_to_ankle" type="fixed">
     <parent link="right_calf" />
@@ -74,4 +89,7 @@
     <xacro:generic_inertia />
   </link>
+  <gazebo reference="right_foot">
+    <material>Gazebo/Blue</material>
+  </gazebo>
   <joint name="right_ankle_to_foot" type="fixed">
     <parent link="right_ankle" />
@@ -83,9 +101,6 @@
         filename="libgazebo_ros_joint_state_publisher.so">
         <update_rate>20</update_rate>
-        <joint_name>base_to_right_hip</joint_name>
         <joint_name>right_hip_to_thigh</joint_name>
-        <joint_name>right_thigh_to_knee</joint_name>
         <joint_name>right_knee_to_calf</joint_name>
-        <joint_name>right_calf_to_ankle</joint_name>
     </plugin>
   </gazebo>
@@ -129,3 +144,23 @@
     </sensor>
   </gazebo>
+  <gazebo reference="right_foot">
+    <gravity>true</gravity>
+    <sensor name="imu_sensor" type="imu">
+      <always_on>true</always_on>
+      <update_rate>100</update_rate>
+      <visualize>true</visualize>
+      <topic>__default_topic__</topic>
+      <plugin filename="libgazebo_ros_imu_sensor.so" name="imu_plugin">
+        <topicName>imu</topicName>
+        <bodyName>right_foot</bodyName>
+        <updateRateHZ>10.0</updateRateHZ>
+        <gaussianNoise>0.0</gaussianNoise>
+        <xyzOffset>0 0 0</xyzOffset>
+        <rpyOffset>0 0 0</rpyOffset>
+        <frameName>right_foot</frameName>
+        <initialOrientationAsReference>false</initialOrientationAsReference>
+      </plugin>
+      <pose>0 0 0 0 0 0</pose>
+    </sensor>
+  </gazebo>
 </robot>

Commit message: motor control?????

File: urdf/model.urdf.xacro (robot description, xacro)
@@ -164,3 +164,25 @@
     </sensor>
   </gazebo>
+  <ros2_control name="GazeboSystem" type="system">
+    <hardware>
+      <plugin>gazebo_ros2_control/GazeboSystem</plugin>
+    </hardware>
+    <joint name="right_knee_to_calf">
+      <command_interface name="effort">
+        <param name="min">-1000</param>
+        <param name="max">1000</param>
+      </command_interface>
+      <state_interface name="position" />
+      <state_interface name="velocity"/>
+      <state_interface name="effort"/>
+    </joint>
+  </ros2_control>
+  <gazebo>
+    <plugin filename="libgazebo_ros2_control.so" name="gazebo_ros2_control">
+      <robot_param>robot_description</robot_param>
+      <robot_param_node>robot_state_publisher</robot_param_node>
+      <parameters>../config/controller.yaml</parameters>
+      <controller_manager_name>controller_manager</controller_manager_name>
+    </plugin>
+  </gazebo>
 </robot>
