Commit message: add second hip joint controller

File: urdf/model.urdf.xacro (robot description, xacro)
@@ -42,5 +42,5 @@
     <origin xyz="${hip_width / 2} 0 0" />
     <axis xyz="1 0 0" rpy="0 0 0"/>
-    <limit lower="${-pi / 2}" upper="${pi / 2}" effort="100" velocity="1" />
+    <limit lower="${-pi / 2}" upper="${pi / 2}" effort="400" velocity="1" />
   </joint>
   <xacro:property name="knee_width" value="0.15" />
@@ -70,5 +70,5 @@
     <origin xyz="0 0 0" />
     <axis xyz="1 0 0" rpy="0 0 0"/>
-    <limit lower="${-pi / 2}" upper="${pi / 2}" effort="100" velocity="1" />
+    <limit lower="${-pi / 2}" upper="${pi / 2}" effort="400" velocity="1" />
   </joint>
   <xacro:property name="ankle_radius" value="0.02" />
@@ -168,4 +168,13 @@
       <plugin>gazebo_ros2_control/GazeboSystem</plugin>
     </hardware>
+    <joint name="right_hip_to_thigh">
+      <command_interface name="effort">
+        <param name="min">-1000</param>
+        <param name="max">1000</param>
+      </command_interface>
+      <state_interface name="position" />
+      <state_interface name="velocity"/>
+      <state_interface name="effort"/>
+    </joint>
     <joint name="right_knee_to_calf">
       <command_interface name="effort">
