Commit message: add calf and lower motor

File: urdf/v2.urdf.xacro (robot description, xacro)
@@ -46,3 +46,69 @@
     <axis xyz="0 1 0" rpy="0 0 0"/>
   </joint>
+  <xacro:property name="thigh_length" value="0.230" />
+  <xacro:property name="thigh_thickness" value="0.0853" />
+  <xacro:property name="thigh_width" value="0.1016" />
+  <link name="left_thigh">
+    <xacro:box_visual_and_collision size="${thigh_length} ${thigh_width} ${thigh_thickness}" xyz="0 0 0" />
+    <xacro:generic_inertia />
+  </link>
+  <joint name="left_motor_to_thigh" type="fixed">
+    <parent link="left_hip_secondary_cylinder" />
+    <child link="left_thigh" />
+    <origin xyz="${thigh_length / 2} 0 0" rpy="0 0 0"/>
+  </joint>
+  <xacro:motor.generate_motor prefix="left_knee" />
+  <joint name="left_thigh_to_knee" type="fixed">
+    <parent link="left_thigh" />
+    <child link="left_knee_primary_cylinder" />
+    <origin xyz="${thigh_length / 2} 0 0" rpy="0 0 0" />
+  </joint>
+  <xacro:property name="calf_plate_length" value="0.100" />
+  <xacro:property name="calf_plate_thickness" value="0.087" />
+  <xacro:property name="calf_plate_width" value="0.0111" />
+  <link name="left_calf_plate">
+    <xacro:box_visual_and_collision size="${calf_plate_length} ${calf_plate_width} ${calf_plate_thickness}" xyz="0 0 0"/>
+    <xacro:generic_inertia />
+  </link>
+  <joint name="left_knee_to_calf" type="revolute">
+    <parent link="left_knee_secondary_cylinder" />
+    <child link="left_calf_plate" />
+    <origin xyz="${calf_plate_length / 2} ${(motor.thickness + calf_plate_width) / 2} 0" rpy="0 0 0" />
+    <limit lower="${-pi / 2}" upper="${pi / 2}" effort="400" velocity="1" />
+    <axis xyz="0 1 0" rpy="0 0 0"/>
+  </joint>
+  <xacro:property name="calf_length" value="0.220" />
+  <xacro:property name="calf_thickness" value="0.0841" />
+  <xacro:property name="calf_width" value="0.059" />
+  <link name="left_calf">
+    <xacro:box_visual_and_collision size="${calf_length} ${calf_width} ${calf_thickness}" xyz="0 0 0" />
+    <xacro:generic_inertia />
+  </link>
+  <joint name="left_calf_plate_to_calf" type="fixed">
+    <parent link="left_calf_plate" />
+    <child link="left_calf" />
+    <origin xyz="${(calf_plate_length + calf_length) / 2} ${-1 * (calf_plate_width + calf_width) / 2} 0" rpy="0 0 0" />
+  </joint>
+  <xacro:property name="ankle_extension_length" value="0.140" />
+  <xacro:property name="ankle_extension_radius" value="0.013" />
+  <link name="left_ankle_extension">
+    <xacro:cylinder_visual_and_collision radius="${ankle_extension_radius}" length="${ankle_extension_length}" xyz="0 0 0" rpy="0 ${pi / 2} 0"/>
+    <xacro:generic_inertia />
+  </link>
+  <joint name="left_calf_to_ankle_extension" type="fixed">
+    <parent link="left_calf" />
+    <child link="left_ankle_extension" />
+    <origin xyz="${(calf_length + ankle_extension_length) / 2} 0 0" rpy="0 0 0" />
+  </joint>
+  <xacro:property name="ankle_length" value="0.035" />
+  <xacro:property name="ankle_radius" value="0.070" />
+  <link name="left_ankle">
+    <xacro:cylinder_visual_and_collision radius="${ankle_radius}" length="${ankle_length}" xyz="0 0 0" rpy="${pi / 2} 0 0" />
+    <xacro:generic_inertia />
+  </link>
+  <joint name="left_ankle_extension_to_ankle" type="fixed">
+    <parent link="left_ankle_extension" />
+    <child link="left_ankle" />
+    <origin xyz="${ankle_extension_length / 2} 0 0" rpy="0 0 0" />
+  </joint>
 </robot>

Commit message: add ankle base

File: urdf/v2.urdf.xacro (robot description, xacro)
@@ -112,3 +112,27 @@
     <origin xyz="${ankle_extension_length / 2} 0 0" rpy="0 0 0" />
   </joint>
+  <xacro:property name="ankle_side_length" value="0.110" />
+  <xacro:property name="ankle_side_thickness" value="0.044" />
+  <xacro:property name="ankle_side_width" value="0.0175" />
+  <link name="left_ankle_side">
+    <xacro:box_visual_and_collision size="${ankle_side_length} ${ankle_side_width} ${ankle_side_thickness}" xyz="0 0 0" />
+    <xacro:generic_inertia />
+  </link>
+  <joint name="left_ankle_to_ankle_side" type="fixed">
+    <parent link="left_ankle" />
+    <child link="left_ankle_side" />
+    <origin xyz="${ankle_side_length / 2} ${(ankle_length + ankle_side_width) / 2} 0" rpy="0 0 0" />
+  </joint>
+  <xacro:property name="ankle_base_length" value="0.3155" />
+  <xacro:property name="ankle_base_width" value="0.120" />
+  <xacro:property name="ankle_base_thickness" value="0.013" />
+  <link name="left_ankle_base">
+    <xacro:box_visual_and_collision size="${ankle_base_thickness} ${ankle_base_width} ${ankle_base_length}" xyz="0 0 0"/>
+    <xacro:generic_inertia />
+  </link>
+  <joint name="left_ankle_side_to_base" type="fixed">
+    <parent link="left_ankle_side" />
+    <child link="left_ankle_base" />
+    <origin xyz="${ankle_side_length / 2} ${ankle_base_width / 2} ${-1 * ankle_base_length / 4}" rpy="0 0 0" />
+  </joint>
 </robot>

Commit message: trying to combine into smaller component

File: urdf/v2.urdf.xacro (robot description, xacro)
@@ -5,4 +5,6 @@
   <xacro:include filename="back.xacro" ns="back" />
   <xacro:include filename="motor.xacro" ns="motor" />
+  <xacro:include filename="calf.xacro" ns="calf" />
+  <xacro:include filename="calf_to_ankle.xacro" ns="calf_to_ankle" />
   <!-- x = left, y = robot back, z = up -->
   <link name="world"></link>
@@ -64,75 +66,11 @@
     <origin xyz="${thigh_length / 2} 0 0" rpy="0 0 0" />
   </joint>
-  <xacro:property name="calf_plate_length" value="0.100" />
-  <xacro:property name="calf_plate_thickness" value="0.087" />
-  <xacro:property name="calf_plate_width" value="0.0111" />
-  <link name="left_calf_plate">
-    <xacro:box_visual_and_collision size="${calf_plate_length} ${calf_plate_width} ${calf_plate_thickness}" xyz="0 0 0"/>
-    <xacro:generic_inertia />
-  </link>
+ <xacro:calf_to_ankle.generate_calf_to_ankle prefix="left" />
   <joint name="left_knee_to_calf" type="revolute">
     <parent link="left_knee_secondary_cylinder" />
     <child link="left_calf_plate" />
-    <origin xyz="${calf_plate_length / 2} ${(motor.thickness + calf_plate_width) / 2} 0" rpy="0 0 0" />
+    <origin xyz="${calf.plate_length / 2} ${(motor.thickness + calf.plate_width) / 2} 0" rpy="0 0 0" />
     <limit lower="${-pi / 2}" upper="${pi / 2}" effort="400" velocity="1" />
     <axis xyz="0 1 0" rpy="0 0 0"/>
   </joint>
-  <xacro:property name="calf_length" value="0.220" />
-  <xacro:property name="calf_thickness" value="0.0841" />
-  <xacro:property name="calf_width" value="0.059" />
-  <link name="left_calf">
-    <xacro:box_visual_and_collision size="${calf_length} ${calf_width} ${calf_thickness}" xyz="0 0 0" />
-    <xacro:generic_inertia />
-  </link>
-  <joint name="left_calf_plate_to_calf" type="fixed">
-    <parent link="left_calf_plate" />
-    <child link="left_calf" />
-    <origin xyz="${(calf_plate_length + calf_length) / 2} ${-1 * (calf_plate_width + calf_width) / 2} 0" rpy="0 0 0" />
-  </joint>
-  <xacro:property name="ankle_extension_length" value="0.140" />
-  <xacro:property name="ankle_extension_radius" value="0.013" />
-  <link name="left_ankle_extension">
-    <xacro:cylinder_visual_and_collision radius="${ankle_extension_radius}" length="${ankle_extension_length}" xyz="0 0 0" rpy="0 ${pi / 2} 0"/>
-    <xacro:generic_inertia />
-  </link>
-  <joint name="left_calf_to_ankle_extension" type="fixed">
-    <parent link="left_calf" />
-    <child link="left_ankle_extension" />
-    <origin xyz="${(calf_length + ankle_extension_length) / 2} 0 0" rpy="0 0 0" />
-  </joint>
-  <xacro:property name="ankle_length" value="0.035" />
-  <xacro:property name="ankle_radius" value="0.070" />
-  <link name="left_ankle">
-    <xacro:cylinder_visual_and_collision radius="${ankle_radius}" length="${ankle_length}" xyz="0 0 0" rpy="${pi / 2} 0 0" />
-    <xacro:generic_inertia />
-  </link>
-  <joint name="left_ankle_extension_to_ankle" type="fixed">
-    <parent link="left_ankle_extension" />
-    <child link="left_ankle" />
-    <origin xyz="${ankle_extension_length / 2} 0 0" rpy="0 0 0" />
-  </joint>
-  <xacro:property name="ankle_side_length" value="0.110" />
-  <xacro:property name="ankle_side_thickness" value="0.044" />
-  <xacro:property name="ankle_side_width" value="0.0175" />
-  <link name="left_ankle_side">
-    <xacro:box_visual_and_collision size="${ankle_side_length} ${ankle_side_width} ${ankle_side_thickness}" xyz="0 0 0" />
-    <xacro:generic_inertia />
-  </link>
-  <joint name="left_ankle_to_ankle_side" type="fixed">
-    <parent link="left_ankle" />
-    <child link="left_ankle_side" />
-    <origin xyz="${ankle_side_length / 2} ${(ankle_length + ankle_side_width) / 2} 0" rpy="0 0 0" />
-  </joint>
-  <xacro:property name="ankle_base_length" value="0.3155" />
-  <xacro:property name="ankle_base_width" value="0.120" />
-  <xacro:property name="ankle_base_thickness" value="0.013" />
-  <link name="left_ankle_base">
-    <xacro:box_visual_and_collision size="${ankle_base_thickness} ${ankle_base_width} ${ankle_base_length}" xyz="0 0 0"/>
-    <xacro:generic_inertia />
-  </link>
-  <joint name="left_ankle_side_to_base" type="fixed">
-    <parent link="left_ankle_side" />
-    <child link="left_ankle_base" />
-    <origin xyz="${ankle_side_length / 2} ${ankle_base_width / 2} ${-1 * ankle_base_length / 4}" rpy="0 0 0" />
-  </joint>
 </robot>
