Commit message: extract thigh

File: urdf/back.xacro (robot description, xacro)
@@ -5,6 +5,10 @@
   <xacro:property name="main_width" value="0.3" />
   <xacro:property name="main_height" value="0.3"/>
+  <xacro:property name="plate_thickness" value="0.005" />
+  <xacro:property name="plate_width" value="0.3" />
+  <xacro:property name="plate_height" value="0.485" />
+  <xacro:property name="rear_spacing" value="0.18" />
   <xacro:macro name="generate_back">
-    <link name="main">
+    <link name="back_main">
       <xacro:box_visual_and_collision size="${main_width} ${main_thickness} ${main_height}" xyz="0 0 0"/>
       <xacro:generic_inertia />
@@ -12,25 +16,15 @@
     <joint name="base_joint" type="fixed">
       <parent link="world"/>
-      <child link="main"/>
-      <origin xyz="0 0 1" rpy="0 0 0"/>
+      <child link="back_main"/>
+      <origin xyz="0 0 1.5" rpy="0 0 0"/>
     </joint>
-    <xacro:property name="plate_thickness" value="0.005" />
-    <xacro:property name="plate_width" value="0.3" />
-    <xacro:property name="plate_height" value="0.485" />
-    <link name="plate">
+    <link name="back_plate">
       <xacro:box_visual_and_collision size="${plate_width} ${plate_thickness} ${plate_height}" xyz="0 0 0"/>
       <xacro:generic_inertia />
     </link>
-    <joint name="plate_joint" type="fixed">
-      <parent link="main"/>
-      <child link="plate"/>
+    <joint name="back_plate_joint" type="fixed">
+      <parent link="back_main"/>
+      <child link="back_plate"/>
       <origin xyz="0 ${-1 * (main_thickness + plate_thickness) / 2} ${-1 * (plate_height - main_height) / 2}" rpy="0 0 0"/>
-    </joint>
-    <xacro:property name="rear_spacing" value="0.18" />
-    <link name="left_connection" />
-    <joint name="left_connection_joint" type="fixed">
-      <parent link="plate" />
-      <child link="left_connection" />
-      <origin xyz="${rear_spacing / 2} ${plate_thickness / 2} ${(-1 * plate_height / 2) + motor.radius}" rpy="0 0 0" />
     </joint>
   </xacro:macro>

File: urdf/calf_to_ankle.xacro (robot description, xacro)
@@ -5,6 +5,6 @@
   <xacro:include filename="ankle.xacro" ns="ankle" />
   <xacro:macro name="generate_calf_to_ankle" params="prefix">
-    <xacro:calf.generate_calf prefix="left" />
-    <xacro:ankle.generate_ankle prefix="left" />
+    <xacro:calf.generate_calf prefix="${prefix}" />
+    <xacro:ankle.generate_ankle prefix="${prefix}" />
     <joint name="${prefix}_calf_to_ankle_extension" type="fixed">
       <parent link="${prefix}_calf" />

File: urdf/old/model.urdf.xacro (robot description, xacro)
@@ -191,5 +191,5 @@
       <robot_param>robot_description</robot_param>
       <robot_param_node>robot_state_publisher</robot_param_node>
-      <parameters>../config/controller.yaml</parameters>
+      <parameters>../config/simple_controller.yaml</parameters>
       <controller_manager_name>controller_manager</controller_manager_name>
     </plugin>

File: urdf/v2.urdf.xacro (robot description, xacro)
@@ -7,4 +7,5 @@
   <xacro:include filename="calf.xacro" ns="calf" />
   <xacro:include filename="calf_to_ankle.xacro" ns="calf_to_ankle" />
+  <xacro:include filename="thigh.xacro" ns="thigh" />
   <!-- x = left, y = robot back, z = up -->
   <link name="world"></link>
@@ -12,7 +13,7 @@
   <xacro:motor.generate_motor prefix="left_rear" />
   <joint name="left_rear_motor" type="revolute">
-    <parent link="left_connection" />
+    <parent link="back_plate" />
     <child link="left_rear_primary_cylinder" />
-    <origin xyz="0 ${motor.thickness / 2} 0" rpy="0 0 0" />
+    <origin xyz="${back.rear_spacing / 2} ${(back.plate_thickness + motor.thickness) / 2} ${(-1 * back.plate_height / 2) + motor.radius}" rpy="0 0 0" />
     <limit lower="${-pi / 2}" upper="${pi / 2}" effort="400" velocity="1" />
     <axis xyz="0 1 0" rpy="0 0 0"/>
@@ -40,5 +41,6 @@
     <origin xyz="${rear_center_to_edge_length / 2 - side_plate_thickness / 2} ${motor.height / 2 - side_plate_length / 2} 0" />
   </joint>
-  <xacro:motor.generate_motor prefix="left_hip"/>
+  <xacro:property name="prefix" value="left" />
+  <xacro:thigh.generate_thigh prefix="${prefix}" />
   <joint name="left_hip_motor" type="revolute">
     <parent link="left_side_plate" />
@@ -48,23 +50,5 @@
     <axis xyz="0 1 0" rpy="0 0 0"/>
   </joint>
-  <xacro:property name="thigh_length" value="0.230" />
-  <xacro:property name="thigh_thickness" value="0.0853" />
-  <xacro:property name="thigh_width" value="0.1016" />
-  <link name="left_thigh">
-    <xacro:box_visual_and_collision size="${thigh_length} ${thigh_width} ${thigh_thickness}" xyz="0 0 0" />
-    <xacro:generic_inertia />
-  </link>
-  <joint name="left_motor_to_thigh" type="fixed">
-    <parent link="left_hip_secondary_cylinder" />
-    <child link="left_thigh" />
-    <origin xyz="${thigh_length / 2} 0 0" rpy="0 0 0"/>
-  </joint>
-  <xacro:motor.generate_motor prefix="left_knee" />
-  <joint name="left_thigh_to_knee" type="fixed">
-    <parent link="left_thigh" />
-    <child link="left_knee_primary_cylinder" />
-    <origin xyz="${thigh_length / 2} 0 0" rpy="0 0 0" />
-  </joint>
- <xacro:calf_to_ankle.generate_calf_to_ankle prefix="left" />
+  <xacro:calf_to_ankle.generate_calf_to_ankle prefix="${prefix}" />
   <joint name="left_knee_to_calf" type="revolute">
     <parent link="left_knee_secondary_cylinder" />
@@ -74,3 +58,12 @@
     <axis xyz="0 1 0" rpy="0 0 0"/>
   </joint>
+   <gazebo>
+      <plugin name="gazebo_ros_joint_state_publisher"
+          filename="libgazebo_ros_joint_state_publisher.so">
+          <update_rate>20</update_rate>
+          <joint_name>left_rear_motor</joint_name>
+          <joint_name>left_hip_motor</joint_name>
+          <joint_name>left_knee_to_calf</joint_name>
+      </plugin>
+    </gazebo>
 </robot>

Commit message: add inertias to components

File: urdf/back.xacro (robot description, xacro)
@@ -11,6 +11,5 @@
   <xacro:macro name="generate_back">
     <link name="back_main">
-      <xacro:box_visual_and_collision size="${main_width} ${main_thickness} ${main_height}" xyz="0 0 0"/>
-      <xacro:generic_inertia />
+      <xacro:box width="${main_width}" depth="${main_thickness}" height="${main_height}" />
     </link>
     <joint name="base_joint" type="fixed">
@@ -20,6 +19,5 @@
     </joint>
     <link name="back_plate">
-      <xacro:box_visual_and_collision size="${plate_width} ${plate_thickness} ${plate_height}" xyz="0 0 0"/>
-      <xacro:generic_inertia />
+      <xacro:box width="${plate_width}" depth="${plate_thickness}" height="${plate_height}" />
     </link>
     <joint name="back_plate_joint" type="fixed">

File: urdf/common.xacro (robot description, xacro)
@@ -1,29 +1,41 @@
 <?xml version="1.0"?>
 <robot xmlns:xacro="http://www.ros.org/wiki/xacro">
-  <xacro:proprety name="zero_transform" value="0 0 0" />
-  <xacro:macro name="generic_inertia">
+  <xacro:property name="zero_transform" value="0 0 0" />
+  <xacro:property name="default_density" value="100" />
+  <xacro:macro name="box" params="width depth height density:=${default_density} xyz:=${zero_transform} color:=red">
+    <xacro:property name="size" value="${width} ${depth} ${height}" />
+    <xacro:property name="volume" value="${width * depth * height}" />
+    <xacro:property name="mass" value="${volume * density}" />
+    <xacro:property name="mass_multiplier" value="${mass / 12}" />
+    <xacro:property name="ixx" value="${mass_multiplier * (depth * depth + height * height)}" />
+    <xacro:property name="iyy" value="${mass_multiplier * (width * width + height * height)}" />
+    <xacro:property name="izz" value="${mass_multiplier * (width * width + depth * depth)}" />
+    <visual>
+      <material name="${color}" />
+      <geometry>
+        <box size="${size}"/>
+      </geometry>
+      <origin xyz="${xyz}" />
+    </visual>
+    <collision>
+      <geometry>
+        <box size="${size}" />
+      </geometry>
+      <origin xyz="${xyz}" />
+    </collision>
     <inertial>
-      <origin xyz="0 0 0" rpy="0 0 0"/>
-      <mass value="12" />
-      <inertia ixx="2.26" ixy="0.0" ixz="0.0" iyy="6.26" iyz="0.0" izz="8.5" />
+      <origin xyz="${xyz}"/>
+      <mass value="${mass}" />
+      <inertia ixx="${ixx}" ixy="0.0" ixz="0.0" iyy="${iyy}" iyz="0.0" izz="${izz}" />
     </inertial>
   </xacro:macro>
-  <xacro:macro name="box" params="depth width height xyz:=${zero_transform} color:=red">
-     <visual>
-        <material name="${color}" />
-        <geometry>
-          <box size="${depth} ${width} ${height}" />
-        </geometry>
-        <origin xyz="${xyz}" />
-      </visual>
-      <collision>
-        <geometry>
-          <box size="${size}" />
-        </geometry>
-        <origin xyz="${xyz}" />
-      </collision>
-  </xacro:macro>
-  <xacro:macro name="cylinder_visual_and_collision" params="length radius xyz rpy color:=red">
-     <visual>
+  <xacro:macro name="cylinder" params="length radius density:=${default_density} xyz:=${zero_transform} rpy:=${zero_transform} color:=red">
+    <xacro:property name="volume" value="${pi * radius * radius * length}" />
+    <xacro:property name="mass" value="${volume * density}" />
+    <xacro:property name="main_inertias" value="${mass / 12 * (3 * radius * radius + length * length)}" />
+    <xacro:property name="ixx" value="${main_inertias}" />
+    <xacro:property name="iyy" value="${main_inertias}" />
+    <xacro:property name="izz" value="${mass / 2 * radius * radius}" />
+    <visual>
       <material name="${color}" />
       <geometry>
@@ -38,4 +50,9 @@
       <origin xyz="${xyz}" rpy="${rpy}"/>
     </collision>
+    <inertial>
+      <origin xyz="${xyz}" rpy="${rpy}"/>
+      <mass value="${mass}" />
+      <inertia ixx="${ixx}" ixy="0.0" ixz="0.0" iyy="${iyy}" iyz="0.0" izz="${izz}" />
+    </inertial>
   </xacro:macro>
 </robot>

File: urdf/leg/ankle.xacro (robot description, xacro)
@@ -14,10 +14,8 @@
   <xacro:macro name="generate_ankle" params="prefix">
     <link name="${prefix}_ankle_extension">
-      <xacro:cylinder_visual_and_collision radius="${extension_radius}" length="${extension_length}" xyz="0 0 0" rpy="0 ${pi / 2} 0"/>
-      <xacro:generic_inertia />
+      <xacro:cylinder radius="${extension_radius}" length="${extension_length}" rpy="0 ${pi / 2} 0" />
     </link>
     <link name="${prefix}_ankle">
-      <xacro:cylinder_visual_and_collision radius="${radius}" length="${length}" xyz="0 0 0" rpy="${pi / 2} 0 0" />
-      <xacro:generic_inertia />
+      <xacro:cylinder radius="${radius}" length="${length}" rpy="${pi / 2} 0 0" />
     </link>
     <joint name="${prefix}_ankle_extension_to_ankle" type="fixed">
@@ -27,6 +25,5 @@
     </joint>
     <link name="${prefix}_ankle_side">
-      <xacro:box_visual_and_collision size="${side_length} ${side_width} ${side_thickness}" xyz="0 0 0" />
-      <xacro:generic_inertia />
+      <xacro:box width="${side_length}" depth="${side_width}" height="${side_thickness}" />
     </link>
     <joint name="${prefix}_ankle_to_ankle_side" type="fixed">
@@ -36,6 +33,5 @@
     </joint>
     <link name="${prefix}_ankle_base">
-      <xacro:box_visual_and_collision size="${base_thickness} ${base_width} ${base_length}" xyz="0 0 0"/>
-      <xacro:generic_inertia />
+      <xacro:box width="${base_thickness}" depth="${base_width}" height="${base_length}" />
     </link>
     <joint name="${prefix}_ankle_side_to_base" type="fixed">

File: urdf/leg/calf.xacro (robot description, xacro)
@@ -10,10 +10,8 @@
   <xacro:macro name="generate_calf" params="prefix">
     <link name="${prefix}_calf_plate">
-      <xacro:box_visual_and_collision size="${plate_length} ${plate_width} ${plate_thickness}" xyz="0 0 0"/>
-      <xacro:generic_inertia />
+      <xacro:box width="${plate_length}" depth="${plate_width}" height="${plate_thickness}" />
     </link>
     <link name="${prefix}_calf">
-      <xacro:box_visual_and_collision size="${length} ${width} ${thickness}" xyz="0 0 0" />
-      <xacro:generic_inertia />
+      <xacro:box width="${length}" depth="${width}" height="${thickness}" />
     </link>
     <joint name="${prefix}_plate_to_calf" type="fixed">

File: urdf/leg/calf_to_ankle.xacro (robot description, xacro)
@@ -1,5 +1,4 @@
 <?xml version="1.0"?>
 <robot xmlns:xacro="http://www.ros.org/wiki/xacro">
-  <xacro:include filename="../common.xacro" />
   <xacro:include filename="calf.xacro" ns="calf"/>
   <xacro:include filename="ankle.xacro" ns="ankle" />

File: urdf/leg/rear_limb.xacro (robot description, xacro)
@@ -10,6 +10,5 @@
     <xacro:motor.generate_motor prefix="${prefix}_rear" />
     <link name="${prefix}_rear_limb">
-      <xacro:box_visual_and_collision size="${rear_center_to_edge_length} ${motor.thickness} ${motor.radius * 2}" xyz="0 0 0"/>
-      <xacro:generic_inertia />
+      <xacro:box width="${rear_center_to_edge_length}" depth="${motor.thickness}" height="${motor.radius * 2}" />
     </link>
     <joint name="${prefix}_rear_limb_to_motor_joint" type="fixed">
@@ -19,6 +18,5 @@
     </joint>
     <link name="${prefix}_side_plate">
-      <xacro:box_visual_and_collision size="${side_plate_thickness} ${side_plate_length} ${side_plate_height}" xyz="0 0 0" />
-      <xacro:generic_inertia />
+      <xacro:box width="${side_plate_thickness}" depth="${side_plate_length}" height="${side_plate_height}" />
     </link>
     <joint name="${prefix}_side_plate_to_rear_limb" type="fixed">

File: urdf/leg/thigh.xacro (robot description, xacro)
@@ -9,6 +9,5 @@
     <xacro:motor.generate_motor prefix="${prefix}_hip"/>
     <link name="${prefix}_thigh">
-      <xacro:box_visual_and_collision size="${length} ${width} ${thickness}" xyz="0 0 0" />
-      <xacro:generic_inertia />
+      <xacro:box width="${length}" depth="${width}" height="${thickness}" />
     </link>
     <joint name="${prefix}_motor_to_thigh" type="fixed">

File: urdf/motor.xacro (robot description, xacro)
@@ -9,8 +9,8 @@
   <xacro:property name="radius" value="${0.120 / 2}" />
   <xacro:property name="inter_center_length" value="${width - 2 * radius}" />
+  <xacro:property name="density" value="1000" />
   <xacro:macro name="single_cylinder" params="name">
     <link name="${name}">
-      <xacro:cylinder_visual_and_collision radius="${radius}" length="${thickness}" xyz="0 0 0" rpy="${pi / 2} 0 0" color="blue"/>
-      <xacro:generic_inertia />
+      <xacro:cylinder radius="${radius}" length="${thickness}" rpy="${pi / 2} 0 0" density="${density}" color="blue" />
     </link>
   </xacro:macro>
@@ -22,6 +22,5 @@
     <!-- a rectangle that shows the connection space between circles -->
     <link name="${prefix}_motor_length">
-      <xacro:box_visual_and_collision size="${inter_center_length} ${thickness} ${height}" xyz="0 0 0" color="blue"/>
-      <xacro:generic_inertia />
+      <xacro:box width="${inter_center_length}" depth="${thickness}" height="${height}" color="blue" density="${density}" />
     </link>
     <joint name="${prefix}_driving_to_length" type="fixed">
