Commit message: found a fix with motor torques

File: urdf/justMotor.urdf.xacro (robot description, xacro)
@@ -6,27 +6,31 @@
   <!-- x = left, y = robot back, z = up -->
   <link name="world"></link>
-  <xacro:motor.generate_motor prefix="main" />
+  <link name="base">
+    <xacro:common.box width="0.2" depth="0.2" height="0.2" density="100" />
+  </link>
   <joint name="fix" type="fixed">
     <parent link="world" />
-    <child link="main_primary_cylinder" />
+    <child link="base" />
     <origin xyz="0 0 0.2" rpy="0 0 0" />
   </joint>
   <link name="propellor">
-    <xacro:common.box width="0.05" depth="0.01" height="0.01" density="100" />
+    <xacro:common.cylinder length="0.1" radius="0.01" density="100" rpy="${pi / 2} 0 0" />
   </link>
   <joint name="propellor_joint" type="revolute">
-    <parent link="main_primary_cylinder" />
+    <parent link="base" />
     <child link="propellor" />
-    <origin xyz="0 ${-1 * motor.thickness} 0" />
+    <origin xyz="0 -0.15 0" />
     <limit lower="${-100 * pi}" upper="${100 * pi}" effort="100000" velocity="1000000" />
     <axis xyz="0 1 0" />
+    <dynamics damping="0.1" friction="0.1" />
   </joint>
-  <gazebo>
-    <plugin name="gazebo_ros_joint_state_publisher"
-        filename="libgazebo_ros_joint_state_publisher.so">
-        <update_rate>100</update_rate>
-        <joint_name>propellor_joint</joint_name>
-    </plugin>
-  </gazebo>
+  <link name="pendulum_mass">
+    <xacro:common.cylinder length="0.3" radius="0.01" density="10000" />
+  </link>
+  <joint name="pendulum_joint" type="fixed">
+    <parent link="propellor" />
+    <child link="pendulum_mass" />
+    <origin xyz="0 -0.05 0.15" />
+  </joint>
   <ros2_control name="GazeboSystem" type="system">
     <hardware>
@@ -45,8 +49,5 @@
   <gazebo>
     <plugin filename="libgazebo_ros2_control.so" name="gazebo_ros2_control">
-      <robot_param>robot_description</robot_param>
-      <robot_param_node>robot_state_publisher</robot_param_node>
       <parameters>../config/motor_controller.yaml</parameters>
-      <controller_manager_name>controller_manager</controller_manager_name>
     </plugin>
   </gazebo>

Commit message: reorganise commandobject

File: urdf/justMotor.urdf.xacro (robot description, xacro)
@@ -12,5 +12,5 @@
     <parent link="world" />
     <child link="base" />
-    <origin xyz="0 0 0.2" rpy="0 0 0" />
+    <origin xyz="0 0 0.5" rpy="0 0 0" />
   </joint>
   <link name="propellor">

Commit message: importing of pid gains

File: urdf/justMotor.urdf.xacro (robot description, xacro)
@@ -23,5 +23,5 @@
     <limit lower="${-100 * pi}" upper="${100 * pi}" effort="100000" velocity="1000000" />
     <axis xyz="0 1 0" />
-    <dynamics damping="0.1" friction="0.1" />
+    <dynamics damping="1" friction="0.1" />
   </joint>
   <link name="pendulum_mass">
