Commit message: define motor macro

File: urdf/common.xacro (robot description, xacro)
@@ -1,4 +1,10 @@
 <?xml version="1.0"?>
 <robot xmlns:xacro="http://www.ros.org/wiki/xacro">
+  <material name="blue">
+    <color rgba="0 0 0.8 1"/>
+  </material>
+  <material name="red">
+    <color rgba="0.8 0 0 1"/>
+  </material>
   <xacro:macro name="generic_inertia">
     <inertial>
@@ -8,6 +14,7 @@
     </inertial>
   </xacro:macro>
-  <xacro:macro name="box_visual_and_collision" params="size xyz">
+  <xacro:macro name="box_visual_and_collision" params="size xyz color:=red">
      <visual>
+        <material name="${color}" />
         <geometry>
           <box size="${size}" />
@@ -22,6 +29,7 @@
       </collision>
   </xacro:macro>
-  <xacro:macro name="cylinder_visual_and_collision" params="length radius xyz rpy">
+  <xacro:macro name="cylinder_visual_and_collision" params="length radius xyz rpy color:=red">
      <visual>
+      <material name="${color}" />
       <geometry>
         <cylinder length="${length}" radius="${radius}" />

File: urdf/v2.urdf.xacro (robot description, xacro)
@@ -1,5 +1,5 @@
 <?xml version="1.0"?>
 <robot name="ALEX_Model_v2" xmlns:xacro="http://www.ros.org/wiki/xacro">
-  <xacro:include filename="common.xacro" />
+  <xacro:include filename="fouriermotor.xacro" />
   <!-- x = left, y = robot back, z = up -->
   <link name="world"></link>
@@ -28,27 +28,34 @@
     <origin xyz="0 ${-1 * (back_plate_thickness + thin_plate_thickness) / 2} ${-1 * (thin_plate_height - back_plate_height) / 2}" rpy="0 0 0"/>
   </joint>
-  <xacro:property name="rear_motor_housing_height" value="0.096"/>
-  <xacro:property name="rear_motor_housing_radius" value="${0.136 / 2}"/>
-  <link name="left_rear">
-    <xacro:cylinder_visual_and_collision radius="${rear_motor_housing_radius}" length="${rear_motor_housing_height}" xyz="0 0 0" rpy="${pi / 2} 0 0"/>
-    <xacro:generic_inertia />
-  </link>
+  <xacro:motor prefix="left_rear" />
   <xacro:property name="rear_spacing" value="0.18" />
-  <joint name="plate_rear_joint" type="revolute">
+  <joint name="left_rear_motor" type="revolute">
     <parent link="thin_plate" />
-    <child link="left_rear" />
-    <origin xyz="${rear_spacing / 2} ${rear_motor_housing_height / 2} ${(-1 * thin_plate_height / 2) + rear_motor_housing_radius}" rpy="0 0 0" />
+    <child link="left_rear_primary_cylinder" />
+    <origin xyz="${rear_spacing / 2} ${motor_thickness / 2} ${(-1 * thin_plate_height / 2) + motor_radius}" rpy="0 0 0" />
     <limit lower="${-pi / 2}" upper="${pi / 2}" effort="400" velocity="1" />
     <axis xyz="0 1 0" rpy="0 0 0"/>
   </joint>
-  <xacro:property name="rear_center_to_edge_length" value="0.240" />
+  <xacro:property name="rear_center_to_edge_length" value="0.130" />
   <link name="left_rear_limb">
-    <xacro:box_visual_and_collision size="${rear_center_to_edge_length} ${rear_motor_housing_height} ${rear_motor_housing_radius * 2}" xyz="0 0 0"/>
+    <xacro:box_visual_and_collision size="${rear_center_to_edge_length} ${motor_thickness} ${motor_radius * 2}" xyz="0 0 0"/>
     <xacro:generic_inertia />
   </link>
   <joint name="left_rear_limb_to_motor_joint" type="fixed">
-    <parent link="left_rear"/>
+    <parent link="left_rear_secondary_cylinder"/>
     <child link="left_rear_limb"/>
     <origin xyz="${rear_center_to_edge_length / 2} 0 0" rpy="0 0 0" />
   </joint>
+  <xacro:property name="side_plate_length" value="0.260" />
+  <xacro:property name="side_plate_height" value="0.06" />
+  <xacro:property name="side_plate_thickness" value="0.028" />
+  <link name="left_side_plate">
+    <xacro:box_visual_and_collision size="${side_plate_thickness} ${side_plate_length} ${side_plate_height}" xyz="0 0 0" />
+    <xacro:generic_inertia />
+  </link>
+  <joint name="left_side_plate_to_rear_limb" type="fixed">
+    <parent link="left_rear_limb" />
+    <child link="left_side_plate" />
+    <origin xyz="${rear_center_to_edge_length / 2 - side_plate_thickness / 2} ${motor_height / 2 - side_plate_length / 2} 0" />
+  </joint>
 </robot>

Commit message: abstract back

File: urdf/common.xacro (robot description, xacro)
@@ -1,10 +1,4 @@
 <?xml version="1.0"?>
 <robot xmlns:xacro="http://www.ros.org/wiki/xacro">
-  <material name="blue">
-    <color rgba="0 0 0.8 1"/>
-  </material>
-  <material name="red">
-    <color rgba="0.8 0 0 1"/>
-  </material>
   <xacro:macro name="generic_inertia">
     <inertial>

File: urdf/motor.xacro (robot description, xacro)
@@ -3,13 +3,13 @@
   <xacro:include filename="common.xacro" />
   <!-- taken from the datasheet -->
-  <xacro:property name="motor_thickness" value="0.075" />
-  <xacro:property name="motor_width" value="0.225" />
-  <xacro:property name="motor_height" value="0.120" />
+  <xacro:property name="thickness" value="0.075" />
+  <xacro:property name="width" value="0.225" />
+  <xacro:property name="height" value="0.120" />
   <!-- calculated values for urdf model -->
-  <xacro:property name="motor_radius" value="${0.120 / 2}" />
-  <xacro:property name="inter_center_length" value="${motor_width - 2 * motor_radius}" />
-  <xacro:macro name="motor_cylinder" params="name">
+  <xacro:property name="radius" value="${0.120 / 2}" />
+  <xacro:property name="inter_center_length" value="${width - 2 * radius}" />
+  <xacro:macro name="single_cylinder" params="name">
     <link name="${name}">
-      <xacro:cylinder_visual_and_collision radius="${motor_radius}" length="${motor_thickness}" xyz="0 0 0" rpy="${pi / 2} 0 0" color="blue"/>
+      <xacro:cylinder_visual_and_collision radius="${radius}" length="${thickness}" xyz="0 0 0" rpy="${pi / 2} 0 0" color="blue"/>
       <xacro:generic_inertia />
     </link>
@@ -17,10 +17,10 @@
   <!-- this macro requires a joint connecting to the ${prefix}_primary_cylinder -->
   <!-- and can connect off the link ${prefix}_secondary_cylinder -->
-  <xacro:macro name="motor" params="prefix">
+  <xacro:macro name="generate_motor" params="prefix">
     <!-- the circle that provides torque -->
-    <xacro:motor_cylinder name="${prefix}_primary_cylinder" />
+    <xacro:single_cylinder name="${prefix}_primary_cylinder" />
     <!-- a rectangle that shows the connection space between circles -->
     <link name="${prefix}_motor_length">
-      <xacro:box_visual_and_collision size="${inter_center_length} ${motor_thickness} ${motor_height}" xyz="0 0 0" color="blue"/>
+      <xacro:box_visual_and_collision size="${inter_center_length} ${thickness} ${height}" xyz="0 0 0" color="blue"/>
       <xacro:generic_inertia />
     </link>
@@ -31,5 +31,5 @@
     </joint>
     <!-- the circle that takes in the Ethernet input -->
-    <xacro:motor_cylinder name="${prefix}_secondary_cylinder" />
+    <xacro:single_cylinder name="${prefix}_secondary_cylinder" />
     <joint name="${prefix}_length_to_signal" type="fixed">
       <parent link="${prefix}_motor_length" />

File: urdf/v2.urdf.xacro (robot description, xacro)
@@ -1,37 +1,16 @@
 <?xml version="1.0"?>
 <robot name="ALEX_Model_v2" xmlns:xacro="http://www.ros.org/wiki/xacro">
-  <xacro:include filename="fouriermotor.xacro" />
+  <xacro:include filename="materials.xacro" />
+  <xacro:include filename="common.xacro" />
+  <xacro:include filename="back.xacro" ns="back" />
+  <xacro:include filename="motor.xacro" ns="motor" />
   <!-- x = left, y = robot back, z = up -->
   <link name="world"></link>
-  <xacro:property name="back_plate_thickness" value="0.08" />
-  <xacro:property name="back_plate_width" value="0.3" />
-  <xacro:property name="back_plate_height" value="0.3"/>
-  <link name="back_plate">
-    <xacro:box_visual_and_collision size="${back_plate_width} ${back_plate_thickness} ${back_plate_height}" xyz="0 0 0"/>
-    <xacro:generic_inertia />
-  </link>
-  <joint name="base_joint" type="fixed">
-    <parent link="world"/>
-    <child link="back_plate"/>
-    <origin xyz="0 0 1" rpy="0 0 0"/>
-  </joint>
-  <xacro:property name="thin_plate_thickness" value="0.005" />
-  <xacro:property name="thin_plate_width" value="0.3" />
-  <xacro:property name="thin_plate_height" value="0.485" />
-  <link name="thin_plate">
-    <xacro:box_visual_and_collision size="${thin_plate_width} ${thin_plate_thickness} ${thin_plate_height}" xyz="0 0 0"/>
-    <xacro:generic_inertia />
-  </link>
-  <joint name="plate_joint" type="fixed">
-    <parent link="back_plate"/>
-    <child link="thin_plate"/>
-    <origin xyz="0 ${-1 * (back_plate_thickness + thin_plate_thickness) / 2} ${-1 * (thin_plate_height - back_plate_height) / 2}" rpy="0 0 0"/>
-  </joint>
-  <xacro:motor prefix="left_rear" />
-  <xacro:property name="rear_spacing" value="0.18" />
+  <xacro:back.generate_back />
+  <xacro:motor.generate_motor prefix="left_rear" />
   <joint name="left_rear_motor" type="revolute">
-    <parent link="thin_plate" />
+    <parent link="left_connection" />
     <child link="left_rear_primary_cylinder" />
-    <origin xyz="${rear_spacing / 2} ${motor_thickness / 2} ${(-1 * thin_plate_height / 2) + motor_radius}" rpy="0 0 0" />
+    <origin xyz="0 ${motor.thickness / 2} 0" rpy="0 0 0" />
     <limit lower="${-pi / 2}" upper="${pi / 2}" effort="400" velocity="1" />
     <axis xyz="0 1 0" rpy="0 0 0"/>
@@ -39,5 +18,5 @@
   <xacro:property name="rear_center_to_edge_length" value="0.130" />
   <link name="left_rear_limb">
-    <xacro:box_visual_and_collision size="${rear_center_to_edge_length} ${motor_thickness} ${motor_radius * 2}" xyz="0 0 0"/>
+    <xacro:box_visual_and_collision size="${rear_center_to_edge_length} ${motor.thickness} ${motor.radius * 2}" xyz="0 0 0"/>
     <xacro:generic_inertia />
   </link>
@@ -57,5 +36,5 @@
     <parent link="left_rear_limb" />
     <child link="left_side_plate" />
-    <origin xyz="${rear_center_to_edge_length / 2 - side_plate_thickness / 2} ${motor_height / 2 - side_plate_length / 2} 0" />
+    <origin xyz="${rear_center_to_edge_length / 2 - side_plate_thickness / 2} ${motor.height / 2 - side_plate_length / 2} 0" />
   </joint>
 </robot>

Commit message: encoder subscriber and start of fixing inertia

File: urdf/common.xacro (robot description, xacro)
@@ -1,4 +1,5 @@
 <?xml version="1.0"?>
 <robot xmlns:xacro="http://www.ros.org/wiki/xacro">
+  <xacro:proprety name="zero_transform" value="0 0 0" />
   <xacro:macro name="generic_inertia">
     <inertial>
@@ -8,9 +9,9 @@
     </inertial>
   </xacro:macro>
-  <xacro:macro name="box_visual_and_collision" params="size xyz color:=red">
+  <xacro:macro name="box" params="depth width height xyz:=${zero_transform} color:=red">
      <visual>
         <material name="${color}" />
         <geometry>
-          <box size="${size}" />
+          <box size="${depth} ${width} ${height}" />
         </geometry>
         <origin xyz="${xyz}" />

File: urdf/v2.urdf.xacro (robot description, xacro)
@@ -21,5 +21,5 @@
       <plugin name="gazebo_ros_joint_state_publisher"
           filename="libgazebo_ros_joint_state_publisher.so">
-          <update_rate>20</update_rate>
+          <update_rate>100</update_rate>
           <joint_name>left_rear_motor</joint_name>
           <joint_name>left_hip_motor</joint_name>

Commit message: reorganize xacro

File: urdf/common.xacro (robot description, xacro)
@@ -3,6 +3,11 @@
   <xacro:property name="zero_transform" value="0 0 0" />
   <xacro:property name="default_density" value="100" />
-  <xacro:macro name="box" params="width depth height density:=${default_density} xyz:=${zero_transform} color:=red">
-    <xacro:property name="size" value="${width} ${depth} ${height}" />
+  <xacro:macro name="box-geom" params="width depth height xyz:=${zero_transform}">
+    <geometry>
+      <box size="${width} ${depth} ${height}" />
+    </geometry>
+    <origin xyz="${xyz}" />
+  </xacro:macro>
+  <xacro:macro name="box-inertial" params="width depth height density:=${default_density} xyz:=${zero_transform}">
     <xacro:property name="volume" value="${width * depth * height}" />
     <xacro:property name="mass" value="${volume * density}" />
@@ -11,17 +16,4 @@
     <xacro:property name="iyy" value="${mass_multiplier * (width * width + height * height)}" />
     <xacro:property name="izz" value="${mass_multiplier * (width * width + depth * depth)}" />
-    <visual>
-      <material name="${color}" />
-      <geometry>
-        <box size="${size}"/>
-      </geometry>
-      <origin xyz="${xyz}" />
-    </visual>
-    <collision>
-      <geometry>
-        <box size="${size}" />
-      </geometry>
-      <origin xyz="${xyz}" />
-    </collision>
     <inertial>
       <origin xyz="${xyz}"/>
@@ -30,5 +22,21 @@
     </inertial>
   </xacro:macro>
-  <xacro:macro name="cylinder" params="length radius density:=${default_density} xyz:=${zero_transform} rpy:=${zero_transform} color:=red">
+  <xacro:macro name="box" params="width depth height density:=${default_density} xyz:=${zero_transform} color:=red">
+    <visual>
+      <material name="${color}" />
+      <xacro:box-geom width="${width}" depth="${depth}" height="${height}" xyz="${xyz}" />
+    </visual>
+    <collision>
+      <xacro:box-geom width="${width}" depth="${depth}" height="${height}" xyz="${xyz}" />
+    </collision>
+    <xacro:box-inertial width="${width}" depth="${depth}" height="${height}" xyz="${xyz}" />
+  </xacro:macro>
+  <xacro:macro name="cylinder-geom" params="length radius xyz:=${zero_transform} rpy:=${zero_transform}">
+    <geometry>
+      <cylinder length="${length}" radius="${radius}" />
+    </geometry>
+    <origin xyz="${xyz}" rpy="${rpy}"/>
+  </xacro:macro>
+  <xacro:macro name="cylinder-inertia" params="length radius density:=${default_density} xyz:=${zero_transform} rpy:=${zero_transform}">
     <xacro:property name="volume" value="${pi * radius * radius * length}" />
     <xacro:property name="mass" value="${volume * density}" />
@@ -37,17 +45,4 @@
     <xacro:property name="iyy" value="${main_inertias}" />
     <xacro:property name="izz" value="${mass / 2 * radius * radius}" />
-    <visual>
-      <material name="${color}" />
-      <geometry>
-        <cylinder length="${length}" radius="${radius}" />
-      </geometry>
-      <origin xyz="${xyz}" rpy="${rpy}"/>
-    </visual>
-    <collision>
-      <geometry>
-        <cylinder length="${length}" radius="${radius}" />
-      </geometry>
-      <origin xyz="${xyz}" rpy="${rpy}"/>
-    </collision>
     <inertial>
       <origin xyz="${xyz}" rpy="${rpy}"/>
@@ -56,3 +51,13 @@
     </inertial>
   </xacro:macro>
+  <xacro:macro name="cylinder" params="length radius density:=${default_density} xyz:=${zero_transform} rpy:=${zero_transform} color:=red">
+    <visual>
+      <material name="${color}" />
+      <xacro:cylinder-geom length="${length}" radius="${radius}" xyz="${xyz}" rpy="${rpy}" />
+    </visual>
+    <collision>
+      <xacro:cylinder-geom length="${length}" radius="${radius}" xyz="${xyz}" rpy="${rpy}" />
+    </collision>
+    <xacro:cylinder-inertia length="${length}" radius="${radius}" density="${density}" xyz="${xyz}" rpy="${rpy}" />
+  </xacro:macro>
 </robot>

File: urdf/twinMotor.urdf.xacro (robot description, xacro)
@@ -42,5 +42,9 @@
   </joint>
   <link name="top_motor_shaft">
-    <xacro:common.cylinder length="0.025" radius="0.01" density="10000" rpy="0 ${pi / 2} 0" />
+    <visual>
+      <material name="blue" />
+      <xacro:common.cylinder-geom length="0.1" radius="0.01" xyz="${0.025/2} 0 ${0.1/2}"/>
+    </visual>
+    <xacro:common.cylinder length="0.025" radius="0.01" density="10000" rpy="0 ${pi / 2} 0"/>
   </link>
   <joint name="top_motor" type="revolute">
@@ -51,12 +55,4 @@
     <axis xyz="-1 0 0" />
     <dynamics damping="1" friction="0.1" />
-  </joint>
-  <link name="top_motor_propellor">
-    <xacro:common.cylinder length="0.1" radius="0.01" density="10000" rpy="0 0 0" />
-  </link>
-  <joint name="propellor_joint" type="fixed">
-    <parent link="top_motor_shaft" />
-    <child link="top_motor_propellor" />
-    <origin xyz="${0.025 / 2} 0 ${0.1 / 2}" rpy="0 0 0"/>
   </joint>
   <ros2_control name="GazeboSystem" type="system">
