Commit message: control from windows client

File: urdf/twinMotor.urdf.xacro (robot description, xacro)
@@ -7,5 +7,5 @@
   <link name="world"></link>
   <link name="base">
-    <xacro:common.box width="0.2" depth="0.2" height="0.05" density="100" />
+    <xacro:common.box width="0.2" depth="0.2" height="0.05" density="10000" />
   </link>
   <joint name="fix" type="fixed">
@@ -15,5 +15,5 @@
   </joint>
   <link name="motor1_base">
-    <xacro:common.box width="0.1" depth="0.1" height="0.1" density="100" />
+    <xacro:common.box width="0.1" depth="0.1" height="0.1" density="10000" />
   </link>
   <joint name="motor1_base_base" type="fixed">
@@ -23,5 +23,5 @@
   </joint>
   <link name="motor1_shaft">
-    <xacro:common.cylinder length="0.025" radius="0.01" density="100" />
+    <xacro:common.cylinder length="0.025" radius="0.01" density="10000" />
   </link>
   <joint name="motor1" type="revolute">
@@ -34,5 +34,5 @@
   </joint>
   <link name="motor2_base">
-    <xacro:common.box width="0.1" depth="0.1" height="0.1" density="100" />
+    <xacro:common.box width="0.1" depth="0.1" height="0.1" density="10000" />
   </link>
   <joint name="motor2_base_motor1_shaft" type="fixed">
@@ -42,5 +42,5 @@
   </joint>
   <link name="motor2_shaft">
-    <xacro:common.cylinder length="0.025" radius="0.01" density="100" rpy="0 ${pi / 2} 0" />
+    <xacro:common.cylinder length="0.025" radius="0.01" density="10000" rpy="0 ${pi / 2} 0" />
   </link>
   <joint name="motor2" type="revolute">
@@ -51,4 +51,12 @@
     <axis xyz="1 0 0" />
     <dynamics damping="1" friction="0.1" />
+  </joint>
+  <link name="motor2_propellor">
+    <xacro:common.cylinder length="0.1" radius="0.01" density="10000" rpy="0 0 0" />
+  </link>
+  <joint name="propellor" type="fixed">
+    <parent link="motor2_shaft" />
+    <child link="motor2_propellor" />
+    <origin xyz="${0.025 / 2} 0 ${0.1 / 2}" rpy="0 0 0"/>
   </joint>
   <ros2_control name="GazeboSystem" type="system">

Commit message: change urdf naming

File: urdf/twinMotor.urdf.xacro (robot description, xacro)
@@ -14,48 +14,48 @@
     <origin xyz="0 0 0.025" rpy="0 0 0" />
   </joint>
-  <link name="motor1_base">
+  <link name="bottom_motor_base">
     <xacro:common.box width="0.1" depth="0.1" height="0.1" density="10000" />
   </link>
-  <joint name="motor1_base_base" type="fixed">
+  <joint name="bottom_motor_base_to_base" type="fixed">
     <parent link="base" />
-    <child link="motor1_base" />
+    <child link="bottom_motor_base" />
     <origin xyz="0 0 0.075" rpy="0 0 0" />
   </joint>
-  <link name="motor1_shaft">
+  <link name="bottom_motor_shaft">
     <xacro:common.cylinder length="0.025" radius="0.01" density="10000" />
   </link>
-  <joint name="motor1" type="revolute">
-    <parent link="motor1_base" />
-    <child link="motor1_shaft" />
+  <joint name="bottom_motor" type="revolute">
+    <parent link="bottom_motor_base" />
+    <child link="bottom_motor_shaft" />
     <origin xyz="0 0 ${0.05 + 0.025/2}" />
     <limit lower="${-100 * pi}" upper="${100 * pi}" effort="100000" velocity="1000000" />
-    <axis xyz="0 0 1" />
+    <axis xyz="0 0 -1" />
     <dynamics damping="1" friction="0.1" />
   </joint>
-  <link name="motor2_base">
+  <link name="top_motor_base">
     <xacro:common.box width="0.1" depth="0.1" height="0.1" density="10000" />
   </link>
-  <joint name="motor2_base_motor1_shaft" type="fixed">
-    <parent link="motor1_shaft" />
-    <child link="motor2_base" />
+  <joint name="top_motor_base_bottom_motor_shaft" type="fixed">
+    <parent link="bottom_motor_shaft" />
+    <child link="top_motor_base" />
     <origin xyz="0 0 ${0.05 + 0.025/2}" rpy="0 0 0" />
   </joint>
-  <link name="motor2_shaft">
+  <link name="top_motor_shaft">
     <xacro:common.cylinder length="0.025" radius="0.01" density="10000" rpy="0 ${pi / 2} 0" />
   </link>
-  <joint name="motor2" type="revolute">
-    <parent link="motor2_base" />
-    <child link="motor2_shaft" />
+  <joint name="top_motor" type="revolute">
+    <parent link="top_motor_base" />
+    <child link="top_motor_shaft" />
     <origin xyz="${0.05 + 0.025/2} 0 0" />
     <limit lower="${-100 * pi}" upper="${100 * pi}" effort="100000" velocity="1000000" />
-    <axis xyz="1 0 0" />
+    <axis xyz="-1 0 0" />
     <dynamics damping="1" friction="0.1" />
   </joint>
-  <link name="motor2_propellor">
+  <link name="top_motor_propellor">
     <xacro:common.cylinder length="0.1" radius="0.01" density="10000" rpy="0 0 0" />
   </link>
-  <joint name="propellor" type="fixed">
-    <parent link="motor2_shaft" />
-    <child link="motor2_propellor" />
+  <joint name="propellor_joint" type="fixed">
+    <parent link="top_motor_shaft" />
+    <child link="top_motor_propellor" />
     <origin xyz="${0.025 / 2} 0 ${0.1 / 2}" rpy="0 0 0"/>
   </joint>
@@ -64,5 +64,5 @@
       <plugin>gazebo_ros2_control/GazeboSystem</plugin>
     </hardware>
-    <joint name="motor1">
+    <joint name="bottom_motor">
       <command_interface name="effort">
         <param name="min">-1000</param>
@@ -73,5 +73,5 @@
       <state_interface name="effort"/>
     </joint>
-    <joint name="motor2">
+    <joint name="top_motor">
       <command_interface name="effort">
         <param name="min">-1000</param>

Commit message: temp fix for velocity pid

File: urdf/twinMotor.urdf.xacro (robot description, xacro)
@@ -4,40 +4,41 @@
   <xacro:include filename="common.xacro" ns="common" />
   <xacro:include filename="materials.xacro" />
+  <xacro:property name="steeldensity" value="7850" />
   <!-- x = left, y = robot back, z = up -->
   <link name="world"></link>
   <link name="base">
-    <xacro:common.box width="0.2" depth="0.2" height="0.05" density="10000" />
+    <xacro:common.box width="0.15" depth="0.15" height="0.015" density="${steeldensity}" />
   </link>
   <joint name="fix" type="fixed">
     <parent link="world" />
     <child link="base" />
-    <origin xyz="0 0 0.025" rpy="0 0 0" />
+    <origin xyz="0 0 ${0.015/2}" rpy="0 0 0" />
   </joint>
   <link name="bottom_motor_base">
-    <xacro:common.box width="0.1" depth="0.1" height="0.1" density="10000" />
+    <xacro:common.cylinder radius="${0.085 / 2}" length="0.07" density="${steeldensity}" />
   </link>
   <joint name="bottom_motor_base_to_base" type="fixed">
     <parent link="base" />
     <child link="bottom_motor_base" />
-    <origin xyz="0 0 0.075" rpy="0 0 0" />
+    <origin xyz="0 0 ${0.015 /2 + 0.08 - 0.07/2} " rpy="0 0 0" />
   </joint>
   <link name="bottom_motor_shaft">
-    <xacro:common.cylinder length="0.025" radius="0.01" density="10000" />
+    <xacro:common.cylinder length="0.04" radius="${0.0275 / 2}" density="${steeldensity}" />
   </link>
   <joint name="bottom_motor" type="revolute">
     <parent link="bottom_motor_base" />
     <child link="bottom_motor_shaft" />
-    <origin xyz="0 0 ${0.05 + 0.025/2}" />
+    <origin xyz="0 0 ${0.07 / 2 + 0.04/2}" />
     <limit lower="${-100 * pi}" upper="${100 * pi}" effort="100000" velocity="1000000" />
     <axis xyz="0 0 -1" />
-    <dynamics damping="1" friction="0.1" />
+    <dynamics damping="0.7" friction="0.01" />
   </joint>
   <link name="top_motor_base">
-    <xacro:common.box width="0.1" depth="0.1" height="0.1" density="10000" />
+    <xacro:common.cylinder radius="${0.085 / 2}" length="0.07" density="${steeldensity}" rpy="0 ${-pi / 2} 0" />
   </link>
   <joint name="top_motor_base_bottom_motor_shaft" type="fixed">
     <parent link="bottom_motor_shaft" />
     <child link="top_motor_base" />
-    <origin xyz="0 0 ${0.05 + 0.025/2}" rpy="0 0 0" />
+    <origin xyz="0 0 ${0.04 / 2 + 0.085/2}" rpy="0 0 0" />
   </joint>
   <link name="top_motor_shaft">
@@ -46,13 +47,13 @@
       <xacro:common.cylinder-geom length="0.1" radius="0.01" xyz="${0.025/2} 0 ${0.1/2}"/>
     </visual>
-    <xacro:common.cylinder length="0.025" radius="0.01" density="10000" rpy="0 ${pi / 2} 0"/>
+    <xacro:common.cylinder length="0.025" radius="0.01" density="${steeldensity}" rpy="0 ${pi / 2} 0"/>
   </link>
   <joint name="top_motor" type="revolute">
     <parent link="top_motor_base" />
     <child link="top_motor_shaft" />
-    <origin xyz="${0.05 + 0.025/2} 0 0" />
+    <origin xyz="${0.07/2 + 0.025/2} 0 0" />
     <limit lower="${-100 * pi}" upper="${100 * pi}" effort="100000" velocity="1000000" />
     <axis xyz="-1 0 0" />
-    <dynamics damping="1" friction="0.1" />
+    <dynamics damping="0.7" friction="0.01" />
   </joint>
   <ros2_control name="GazeboSystem" type="system">

Commit message: recreation as two large components with meshes

File: urdf/twinMotor.urdf.xacro (robot description, xacro)
@@ -15,4 +15,43 @@
     <origin xyz="0 0 ${0.015/2}" rpy="0 0 0" />
   </joint>
+  <link name="bottom_motor_link">
+    <visual>
+      <xacro:common.cylinder-geom length="0.07" radius="${0.085 / 2}"/>
+    </visual>
+    <collision>
+      <xacro:common.cylinder-geom length="0.07" radius="${0.085 / 2}"/>
+    </collision>
+    <xacro:common.cylinder-inertia length="0.07" radius="${0.085 / 2}" density="${steeldensity}" />
+  </link>
+  <joint name="bottom_motor" type="revolute">
+    <parent link="base" />
+    <child link="bottom_motor_link" />
+    <origin xyz="0 0 ${(0.07 + 0.015)/ 2}" />
+    <limit lower="${-100 * pi}" upper="${100 * pi}" effort="100000" velocity="1000000" />
+    <axis xyz="0 0 -1" />
+  </joint>
+  <link name="top_motor_link">
+    <visual>
+      <xacro:common.cylinder-geom length="0.03" radius="0.03" rpy="0 ${pi / 2} 0" xyz="0.05 0 0"/>
+    </visual>
+    <visual>
+      <xacro:common.cylinder-geom length="0.1" radius="0.01" rpy="0 0 0" xyz="0.05 0 0.05"/>
+    </visual>
+    <visual>
+      <xacro:common.cylinder-geom length="0.07" radius="${0.085 / 2}" rpy="0 ${pi / 2} 0"/>
+    </visual>
+    <collision>
+      <xacro:common.cylinder-geom length="0.07" radius="${0.085 / 2}" rpy="0 ${pi / 2} 0"/>
+    </collision>
+    <xacro:common.cylinder-inertia length="0.07" radius="${0.085 / 2}" density="${steeldensity}" rpy="0 ${pi / 2} 0" />
+  </link>
+  <joint name="top_motor" type="revolute">
+    <parent link="bottom_motor_link" />
+    <child link="top_motor_link" />
+    <origin xyz="0 0 ${0.07 + 0.03}" />
+    <limit lower="${-100 * pi}" upper="${100 * pi}" effort="100000" velocity="1000000" />
+    <axis xyz="1 0 0" />
+  </joint>
+<!--
   <link name="bottom_motor_base">
     <xacro:common.cylinder radius="${0.085 / 2}" length="0.07" density="${steeldensity}" />
@@ -56,5 +95,5 @@
     <axis xyz="-1 0 0" />
     <dynamics damping="0.7" friction="0.01" />
-  </joint>
+  </joint> -->
   <ros2_control name="GazeboSystem" type="system">
     <hardware>

Commit message: delete old urdf

File: urdf/twinMotor.urdf.xacro (robot description, xacro)
@@ -53,47 +53,4 @@
     <axis xyz="1 0 0" />
   </joint>
-<!--
-  <link name="bottom_motor_base">
-    <xacro:common.cylinder radius="${0.085 / 2}" length="0.07" density="${steeldensity}" />
-  </link>
-  <joint name="bottom_motor_base_to_base" type="fixed">
-    <parent link="base" />
-    <child link="bottom_motor_base" />
-    <origin xyz="0 0 ${0.015 /2 + 0.08 - 0.07/2} " rpy="0 0 0" />
-  </joint>
-  <link name="bottom_motor_shaft">
-    <xacro:common.cylinder length="0.04" radius="${0.0275 / 2}" density="${10 * steeldensity}" />
-  </link>
-  <joint name="bottom_motor" type="revolute">
-    <parent link="bottom_motor_base" />
-    <child link="bottom_motor_shaft" />
-    <origin xyz="0 0 ${0.07 / 2 + 0.04/2}" />
-    <limit lower="${-100 * pi}" upper="${100 * pi}" effort="100000" velocity="1000000" />
-    <axis xyz="0 0 -1" />
-    <dynamics damping="0.7" friction="0.01" />
-  </joint>
-  <link name="top_motor_base">
-    <xacro:common.cylinder radius="${0.085 / 2}" length="0.07" density="${10 * steeldensity}" rpy="0 ${-pi / 2} 0" />
-  </link>
-  <joint name="top_motor_base_bottom_motor_shaft" type="fixed">
-    <parent link="bottom_motor_shaft" />
-    <child link="top_motor_base" />
-    <origin xyz="0 0 ${0.04 / 2 + 0.085/2}" rpy="0 0 0" />
-  </joint>
-  <link name="top_motor_shaft">
-    <visual>
-      <material name="blue" />
-      <xacro:common.cylinder-geom length="0.1" radius="0.01" xyz="${0.025/2} 0 ${0.1/2}"/>
-    </visual>
-    <xacro:common.cylinder length="0.025" radius="0.1" density="${10 * steeldensity}" rpy="0 ${pi / 2} 0"/>
-  </link>
-  <joint name="top_motor" type="revolute">
-    <parent link="top_motor_base" />
-    <child link="top_motor_shaft" />
-    <origin xyz="${0.07/2 + 0.025/2} 0 0" />
-    <limit lower="${-100 * pi}" upper="${100 * pi}" effort="100000" velocity="1000000" />
-    <axis xyz="-1 0 0" />
-    <dynamics damping="0.7" friction="0.01" />
-  </joint> -->
   <ros2_control name="GazeboSystem" type="system">
     <hardware>

Commit message: testing damping

File: urdf/twinMotor.urdf.xacro (robot description, xacro)
@@ -52,4 +52,5 @@
     <limit lower="${-100 * pi}" upper="${100 * pi}" effort="100000" velocity="1000000" />
     <axis xyz="1 0 0" />
+    <dynamics damping="0.15"/>
   </joint>
   <ros2_control name="GazeboSystem" type="system">

Commit message: can run chirp on simulation

File: urdf/twinMotor.urdf.xacro (robot description, xacro)
@@ -52,5 +52,5 @@
     <limit lower="${-100 * pi}" upper="${100 * pi}" effort="100000" velocity="1000000" />
     <axis xyz="1 0 0" />
-    <dynamics damping="0.15"/>
+    <dynamics damping="0.1"/>
   </joint>
   <ros2_control name="GazeboSystem" type="system">

Commit message: flatten folder structure

File: urdf/twinMotor.urdf.xacro (robot description, xacro)
@@ -52,5 +52,5 @@
     <limit lower="${-100 * pi}" upper="${100 * pi}" effort="100000" velocity="1000000" />
     <axis xyz="1 0 0" />
-    <dynamics damping="0.1"/>
+    <dynamics damping="0.5"/>
   </joint>
   <ros2_control name="GazeboSystem" type="system">

Commit message: change sizing of motor urdf

File: urdf/twinMotor.urdf.xacro (robot description, xacro)
@@ -5,4 +5,12 @@
   <xacro:include filename="materials.xacro" />
   <xacro:property name="steeldensity" value="7850" />
+  <xacro:property name="motor_diameter" value="0.085" />
+  <xacro:property name="motor_length" value="0.075" />
+  <xacro:property name="inner_diameter" value="0.06" />
+  <xacro:property name="inner_length" value="0.055" />
+  <xacro:property name="base_length" value="0.09" />
+  <xacro:property name="attachment_height" value="0.035" />
+  <xacro:property name="attachment_diameter" value="0.025" />
+  <xacro:property name="motor_offset" value="${-base_length / 2 + motor_length - inner_length / 2}" />
   <!-- x = left, y = robot back, z = up -->
   <link name="world"></link>
@@ -15,23 +23,29 @@
     <origin xyz="0 0 ${0.015/2}" rpy="0 0 0" />
   </joint>
+  <gazebo reference="bottom_motor_link">
+    <material>Gazebo/Blue</material>
+  </gazebo>
   <link name="bottom_motor_link">
     <visual>
-      <xacro:common.cylinder-geom length="0.07" radius="${0.085 / 2}"/>
+      <xacro:common.cylinder-geom length="${inner_length}" radius="${inner_diameter / 2}"/>
     </visual>
     <collision>
-      <xacro:common.cylinder-geom length="0.07" radius="${0.085 / 2}"/>
+      <xacro:common.cylinder-geom length="${inner_length}" radius="${inner_diameter / 2}"/>
     </collision>
-    <xacro:common.cylinder-inertia length="0.07" radius="${0.085 / 2}" density="${steeldensity}" />
+    <xacro:common.cylinder-inertia length="${inner_length}" radius="${inner_diameter / 2}" density="${steeldensity}" />
   </link>
   <joint name="bottom_motor" type="revolute">
     <parent link="base" />
     <child link="bottom_motor_link" />
-    <origin xyz="0 0 ${(0.07 + 0.015)/ 2}" />
+    <origin xyz="0 0 ${(inner_length + 0.015)/ 2}" />
     <limit lower="${-100 * pi}" upper="${100 * pi}" effort="100000" velocity="1000000" />
     <axis xyz="0 0 -1" />
   </joint>
+  <gazebo reference="top_motor_link">
+    <material>Gazebo/Blue</material>
+  </gazebo>
   <link name="top_motor_link">
     <visual>
-      <xacro:common.cylinder-geom length="0.03" radius="0.03" rpy="0 ${pi / 2} 0" xyz="0.05 0 0"/>
+      <xacro:common.cylinder-geom length="0.03" radius="0.02" rpy="0 ${pi / 2} 0" xyz="0.05 0 0"/>
     </visual>
     <visual>
@@ -39,15 +53,15 @@
     </visual>
     <visual>
-      <xacro:common.cylinder-geom length="0.07" radius="${0.085 / 2}" rpy="0 ${pi / 2} 0"/>
+      <xacro:common.cylinder-geom length="${inner_length}" radius="${inner_length / 2}" rpy="0 ${pi / 2} 0"/>
     </visual>
     <collision>
-      <xacro:common.cylinder-geom length="0.07" radius="${0.085 / 2}" rpy="0 ${pi / 2} 0"/>
+      <xacro:common.cylinder-geom length="${inner_length}" radius="${inner_length / 2}" rpy="0 ${pi / 2} 0"/>
     </collision>
-    <xacro:common.cylinder-inertia length="0.07" radius="${0.085 / 2}" density="${steeldensity}" rpy="0 ${pi / 2} 0" />
+    <xacro:common.cylinder-inertia length="${inner_length}" radius="${inner_length / 2}" density="${steeldensity}" rpy="0 ${pi / 2} 0" />
   </link>
   <joint name="top_motor" type="revolute">
     <parent link="bottom_motor_link" />
     <child link="top_motor_link" />
-    <origin xyz="0 0 ${0.07 + 0.03}" />
+    <origin xyz="${-motor_offset} 0 ${inner_length + attachment_height}" />
     <limit lower="${-100 * pi}" upper="${100 * pi}" effort="100000" velocity="1000000" />
     <axis xyz="1 0 0" />

Commit message: inertia values are too small

File: urdf/twinMotor.urdf.xacro (robot description, xacro)
@@ -38,7 +38,8 @@
     <parent link="base" />
     <child link="bottom_motor_link" />
-    <origin xyz="0 0 ${(inner_length + 0.015)/ 2}" />
+    <origin xyz="0 0 ${(inner_length + 0.02)/ 2}" />
     <limit lower="${-100 * pi}" upper="${100 * pi}" effort="100000" velocity="1000000" />
     <axis xyz="0 0 -1" />
+    <dynamics damping="0.1" friction="0.0"/>
   </joint>
   <gazebo reference="top_motor_link">
@@ -58,5 +59,5 @@
       <xacro:common.cylinder-geom length="${inner_length}" radius="${inner_length / 2}" rpy="0 ${pi / 2} 0"/>
     </collision>
-    <xacro:common.cylinder-inertia length="${inner_length}" radius="${inner_length / 2}" density="${steeldensity}" rpy="0 ${pi / 2} 0" />
+    <xacro:common.cylinder-inertia length="${inner_length}" radius="${inner_length / 2}" density="${20 * steeldensity}" rpy="0 ${pi / 2} 0" />
   </link>
   <joint name="top_motor" type="revolute">
@@ -64,7 +65,7 @@
     <child link="top_motor_link" />
     <origin xyz="${-motor_offset} 0 ${inner_length + attachment_height}" />
-    <limit lower="${-100 * pi}" upper="${100 * pi}" effort="100000" velocity="1000000" />
+    <limit lower="${-100 * pi}" upper="${100 * pi}" effort="100" velocity="100" />
     <axis xyz="1 0 0" />
-    <dynamics damping="0.5"/>
+    <dynamics damping="5" friction="0.0"/>
   </joint>
   <ros2_control name="GazeboSystem" type="system">

Commit message: [yz]: simple steps + damping

File: urdf/twinMotor.urdf.xacro (robot description, xacro)
@@ -41,5 +41,5 @@
     <limit lower="${-100 * pi}" upper="${100 * pi}" effort="100000" velocity="1000000" />
     <axis xyz="0 0 -1" />
-    <dynamics damping="0.1" friction="0.0"/>
+    <dynamics damping="0.0" friction="0.0"/>
   </joint>
   <gazebo reference="top_motor_link">
@@ -59,5 +59,5 @@
       <xacro:common.cylinder-geom length="${inner_length}" radius="${inner_length / 2}" rpy="0 ${pi / 2} 0"/>
     </collision>
-    <xacro:common.cylinder-inertia length="${inner_length}" radius="${inner_length / 2}" density="${20 * steeldensity}" rpy="0 ${pi / 2} 0" />
+    <xacro:common.cylinder-inertia length="${inner_length}" radius="${inner_length / 2}" density="${steeldensity}" rpy="0 ${pi / 2} 0" />
   </link>
   <joint name="top_motor" type="revolute">
@@ -65,7 +65,7 @@
     <child link="top_motor_link" />
     <origin xyz="${-motor_offset} 0 ${inner_length + attachment_height}" />
-    <limit lower="${-100 * pi}" upper="${100 * pi}" effort="100" velocity="100" />
+    <limit lower="${-1000 * pi}" upper="${1000 * pi}" effort="10000" velocity="10000" />
     <axis xyz="1 0 0" />
-    <dynamics damping="5" friction="0.0"/>
+    <dynamics damping="0.001" friction="0.0"/>
   </joint>
   <ros2_control name="GazeboSystem" type="system">

Commit message: [yz]: good selection of friction epsilon term

File: urdf/twinMotor.urdf.xacro (robot description, xacro)
@@ -41,5 +41,5 @@
     <limit lower="${-100 * pi}" upper="${100 * pi}" effort="100000" velocity="1000000" />
     <axis xyz="0 0 -1" />
-    <dynamics damping="0.0" friction="0.0"/>
+    <dynamics damping="0.0" friction="0.05"/>
   </joint>
   <gazebo reference="top_motor_link">
@@ -54,10 +54,10 @@
     </visual>
     <visual>
-      <xacro:common.cylinder-geom length="${inner_length}" radius="${inner_length / 2}" rpy="0 ${pi / 2} 0"/>
+      <xacro:common.cylinder-geom length="${inner_length}" radius="${inner_diameter / 2}" rpy="0 ${pi / 2} 0"/>
     </visual>
     <collision>
-      <xacro:common.cylinder-geom length="${inner_length}" radius="${inner_length / 2}" rpy="0 ${pi / 2} 0"/>
+      <xacro:common.cylinder-geom length="${inner_length}" radius="${inner_diameter / 2}" rpy="0 ${pi / 2} 0"/>
     </collision>
-    <xacro:common.cylinder-inertia length="${inner_length}" radius="${inner_length / 2}" density="${steeldensity}" rpy="0 ${pi / 2} 0" />
+    <xacro:common.cylinder-inertia length="${inner_length}" radius="${inner_diameter / 2}" density="${steeldensity}" rpy="0 ${pi / 2} 0" />
   </link>
   <joint name="top_motor" type="revolute">
@@ -67,5 +67,5 @@
     <limit lower="${-1000 * pi}" upper="${1000 * pi}" effort="10000" velocity="10000" />
     <axis xyz="1 0 0" />
-    <dynamics damping="0.001" friction="0.0"/>
+    <dynamics damping="0.01" friction="0.0999"/>
   </joint>
   <ros2_control name="GazeboSystem" type="system">

Commit message: not sure why position control is no longer working

File: urdf/twinMotor.urdf.xacro (robot description, xacro)
@@ -41,5 +41,5 @@
     <limit lower="${-100 * pi}" upper="${100 * pi}" effort="100000" velocity="1000000" />
     <axis xyz="0 0 -1" />
-    <dynamics damping="0.0" friction="0.05"/>
+    <!-- <dynamics damping="0.0" friction="0.00"/> -->
   </joint>
   <gazebo reference="top_motor_link">
@@ -67,5 +67,5 @@
     <limit lower="${-1000 * pi}" upper="${1000 * pi}" effort="10000" velocity="10000" />
     <axis xyz="1 0 0" />
-    <dynamics damping="0.01" friction="0.0999"/>
+    <!-- <dynamics damping="0.00" friction="0.00"/> -->
   </joint>
   <ros2_control name="GazeboSystem" type="system">

Commit message: looks like damping was too small - issues with time delay

File: urdf/twinMotor.urdf.xacro (robot description, xacro)
@@ -41,5 +41,5 @@
     <limit lower="${-100 * pi}" upper="${100 * pi}" effort="100000" velocity="1000000" />
     <axis xyz="0 0 -1" />
-    <!-- <dynamics damping="0.0" friction="0.00"/> -->
+    <dynamics damping="1" friction="0.00"/>
   </joint>
   <gazebo reference="top_motor_link">
@@ -67,5 +67,5 @@
     <limit lower="${-1000 * pi}" upper="${1000 * pi}" effort="10000" velocity="10000" />
     <axis xyz="1 0 0" />
-    <!-- <dynamics damping="0.00" friction="0.00"/> -->
+    <dynamics damping="1" friction="0.00"/>
   </joint>
   <ros2_control name="GazeboSystem" type="system">
