Commit message: looks like its just because P gain was too high

File: urdf/twinMotor.urdf.xacro (robot description, xacro)
@@ -41,5 +41,5 @@
     <limit lower="${-100 * pi}" upper="${100 * pi}" effort="100000" velocity="1000000" />
     <axis xyz="0 0 -1" />
-    <dynamics damping="1" friction="0.00"/>
+    <dynamics damping="0.01" friction="0.00"/>
   </joint>
   <gazebo reference="top_motor_link">
@@ -67,5 +67,5 @@
     <limit lower="${-1000 * pi}" upper="${1000 * pi}" effort="10000" velocity="10000" />
     <axis xyz="1 0 0" />
-    <dynamics damping="1" friction="0.00"/>
+    <dynamics damping="0.01" friction="0.00"/>
   </joint>
   <ros2_control name="GazeboSystem" type="system">

Commit message: bulk data collection

File: urdf/twinMotor.urdf.xacro (robot description, xacro)
@@ -41,5 +41,5 @@
     <limit lower="${-100 * pi}" upper="${100 * pi}" effort="100000" velocity="1000000" />
     <axis xyz="0 0 -1" />
-    <dynamics damping="0.01" friction="0.00"/>
+    <dynamics damping="0.01" friction="0.05"/>
   </joint>
   <gazebo reference="top_motor_link">
@@ -67,5 +67,5 @@
     <limit lower="${-1000 * pi}" upper="${1000 * pi}" effort="10000" velocity="10000" />
     <axis xyz="1 0 0" />
-    <dynamics damping="0.01" friction="0.00"/>
+    <dynamics damping="0.01" friction="0.05"/>
   </joint>
   <ros2_control name="GazeboSystem" type="system">
