Commit message: completed urdf

File: urdf/exov3.urdf.xacro (robot description, xacro)
@@ -5,5 +5,4 @@
   <xacro:include filename="materials.xacro" />
   <xacro:property name="steeldensity" value="7850" />
-  <!-- x = left, y = robot back, z = up -->
   <link name="world"></link>
   <link name="base">
@@ -64,56 +63,6 @@
     <axis xyz="0 -1 0" />
   </joint>
-<!--
-  <gazebo reference="bottom_motor_link">
-    <material>Gazebo/Blue</material>
-  </gazebo>
-  <link name="back_left_motor_link">
-    <visual>
-      <xacro:common.cylinder-geom length="${inner_length}" radius="${inner_diameter / 2}"/>
-    </visual>
-    <collision>
-      <xacro:common.cylinder-geom length="${inner_length}" radius="${inner_diameter / 2}"/>
-    </collision>
-    <xacro:common.cylinder-inertia length="${inner_length}" radius="${inner_diameter / 2}" density="${steeldensity}" />
-  </link>
-  <joint name="bottom_motor" type="revolute">
-    <parent link="base" />
-    <child link="bottom_motor_link" />
-    <origin xyz="0 0 ${(inner_length + 0.02)/ 2}" />
-    <limit lower="${-100 * pi}" upper="${100 * pi}" effort="100000" velocity="1000000" />
-    <axis xyz="0 0 -1" />
-    <dynamics damping="0.01" friction="0.05"/>
-  </joint>
-  <gazebo reference="top_motor_link">
-    <material>Gazebo/Blue</material>
-  </gazebo>
-  <link name="top_motor_link">
-    <visual>
-      <xacro:common.cylinder-geom length="0.03" radius="0.02" rpy="0 ${pi / 2} 0" xyz="0.05 0 0"/>
-    </visual>
-    <visual>
-      <xacro:common.cylinder-geom length="0.1" radius="0.01" rpy="0 0 0" xyz="0.05 0 0.05"/>
-    </visual>
-    <visual>
-      <xacro:common.cylinder-geom length="${inner_length}" radius="${inner_diameter / 2}" rpy="0 ${pi / 2} 0"/>
-    </visual>
-    <collision>
-      <xacro:common.cylinder-geom length="${inner_length}" radius="${inner_diameter / 2}" rpy="0 ${pi / 2} 0"/>
-    </collision>
-    <xacro:common.cylinder-inertia length="${inner_length}" radius="${inner_diameter / 2}" density="${steeldensity}" rpy="0 ${pi / 2} 0" />
-  </link>
-  <joint name="top_motor" type="revolute">
-    <parent link="bottom_motor_link" />
-    <child link="top_motor_link" />
-    <origin xyz="${-motor_offset} 0 ${inner_length + attachment_height}" />
-    <limit lower="${-1000 * pi}" upper="${1000 * pi}" effort="10000" velocity="10000" />
-    <axis xyz="1 0 0" />
-    <dynamics damping="0.01" friction="0.05"/>
-  </joint>
-  <ros2_control name="GazeboSystem" type="system">
-    <hardware>
-      <plugin>gazebo_ros2_control/GazeboSystem</plugin>
-    </hardware>
-    <joint name="bottom_motor">
+  <xacro:macro name="ros2control_motor" params="name">
+    <joint name="${name}">
       <command_interface name="effort">
         <param name="min">-1000</param>
@@ -124,18 +73,20 @@
       <state_interface name="effort"/>
     </joint>
-    <joint name="top_motor">
-      <command_interface name="effort">
-        <param name="min">-1000</param>
-        <param name="max">1000</param>
-      </command_interface>
-      <state_interface name="position" />
-      <state_interface name="velocity"/>
-      <state_interface name="effort"/>
-    </joint>
+  </xacro:macro>
+  <ros2_control name="GazeboSystem" type="system">
+    <hardware>
+      <plugin>gazebo_ros2_control/GazeboSystem</plugin>
+    </hardware>
+    <xacro:ros2control_motor name="left_abduction"/>
+    <xacro:ros2control_motor name="left_hip"/>
+    <xacro:ros2control_motor name="left_knee"/>
+    <xacro:ros2control_motor name="right_abduction"/>
+    <xacro:ros2control_motor name="right_hip"/>
+    <xacro:ros2control_motor name="right_knee"/>
   </ros2_control>
   <gazebo>
     <plugin filename="libgazebo_ros2_control.so" name="gazebo_ros2_control">
-      <parameters>../config/twin_controller.yaml</parameters>
+      <parameters>../config/exo_controller.yaml</parameters>
     </plugin>
-  </gazebo> -->
+  </gazebo>
 </robot>

Commit message: adequate parameters for fixed state

File: urdf/exov3.urdf.xacro (robot description, xacro)
@@ -5,4 +5,7 @@
   <xacro:include filename="materials.xacro" />
   <xacro:property name="steeldensity" value="7850" />
+  <xacro:macro name="motor_dynamics">
+      <dynamics damping="20" friction="0.5" />
+  </xacro:macro>
   <link name="world"></link>
   <link name="base">
@@ -27,4 +30,5 @@
       <limit lower="${-pi}" upper="${pi}" effort="100" velocity="100" />
       <axis xyz="1 0 0" />
+      <xacro:motor_dynamics />
     </joint>
     <link name="${prefix}_knee_link">
@@ -37,4 +41,5 @@
       <limit lower="${-pi}" upper="${pi}" effort="100" velocity="100" />
       <axis xyz="1 0 0" />
+      <xacro:motor_dynamics />
     </joint>
     <link name="${prefix}_calf_link">
@@ -54,4 +59,5 @@
     <limit lower="${-pi / 2}" upper="${pi / 2}" effort="100" velocity="100" />
     <axis xyz="0 -1 0" />
+    <xacro:motor_dynamics />
   </joint>
   <xacro:leg prefix="right" multiplier="-1" />
@@ -62,4 +68,5 @@
     <limit lower="${-pi / 2}" upper="${pi / 2}" effort="100" velocity="100" />
     <axis xyz="0 -1 0" />
+    <xacro:motor_dynamics />
   </joint>
   <xacro:macro name="ros2control_motor" params="name">

Commit message: maybe the right directions?

File: urdf/exov3.urdf.xacro (robot description, xacro)
@@ -29,5 +29,5 @@
       <origin xyz="${multiplier * 0.2} -0.2 0" rpy="0 0 0" />
       <limit lower="${-pi}" upper="${pi}" effort="100" velocity="100" />
-      <axis xyz="1 0 0" />
+      <axis xyz="${multiplier * -1} 0 0" />
       <xacro:motor_dynamics />
     </joint>
@@ -40,5 +40,5 @@
       <origin xyz="0 0 -0.5" rpy="0 0 0" />
       <limit lower="${-pi}" upper="${pi}" effort="100" velocity="100" />
-      <axis xyz="1 0 0" />
+      <axis xyz="${multiplier * -1} 0 0" />
       <xacro:motor_dynamics />
     </joint>
@@ -86,8 +86,8 @@
     </hardware>
     <xacro:ros2control_motor name="left_abduction"/>
+    <xacro:ros2control_motor name="right_abduction"/>
     <xacro:ros2control_motor name="left_hip"/>
+    <xacro:ros2control_motor name="right_hip"/>
     <xacro:ros2control_motor name="left_knee"/>
-    <xacro:ros2control_motor name="right_abduction"/>
-    <xacro:ros2control_motor name="right_hip"/>
     <xacro:ros2control_motor name="right_knee"/>
   </ros2_control>

Commit message: stability by adding saturation velocities

File: urdf/exov3.urdf.xacro (robot description, xacro)
@@ -6,5 +6,5 @@
   <xacro:property name="steeldensity" value="7850" />
   <xacro:macro name="motor_dynamics">
-      <dynamics damping="20" friction="0.5" />
+      <dynamics damping="0" friction="10.4160" />
   </xacro:macro>
   <link name="world"></link>
@@ -17,10 +17,30 @@
     <origin xyz="0 0 1.5" rpy="0 0 0" />
   </joint>
+  <xacro:macro name="motor_cylinder" params="rpy">
+    <visual>
+      <material name="red" />
+      <geometry>
+        <cylinder length="0.05" radius="0.07" />
+      </geometry>
+      <origin rpy="${rpy}"/>
+    </visual>
+    <collision>
+      <geometry>
+        <cylinder length="0.05" radius="0.07" />
+      </geometry>
+      <origin rpy="${rpy}"/>
+    </collision>
+    <inertial>
+      <origin rpy="${rpy}"/>
+      <mass value="4" />
+      <inertia ixx="0.1" ixy="0.0" ixz="0.0" iyy="0.1" iyz="0.0" izz="9.1617" />
+    </inertial>
+  </xacro:macro>
   <xacro:macro name="leg" params="prefix multiplier">
     <link name="${prefix}_abduction_link">
-      <xacro:common.cylinder radius="0.07" length="0.05" density="${steeldensity}" rpy="${pi / 2} 0 0"/>
+      <xacro:motor_cylinder rpy="${pi / 2} 0 0"/>
     </link>
     <link name="${prefix}_hip_link">
-      <xacro:common.cylinder radius="0.07" length="0.05" density="${steeldensity}" rpy="0 ${pi / 2} 0"/>
+      <xacro:motor_cylinder rpy="0 ${pi / 2} 0"/>
     </link>
     <joint name="${prefix}_hip" type="revolute">
@@ -33,5 +53,5 @@
     </joint>
     <link name="${prefix}_knee_link">
-      <xacro:common.cylinder radius="0.07" length="0.05" density="${steeldensity}" rpy="0 ${pi / 2} 0"/>
+      <xacro:motor_cylinder rpy="0 ${pi / 2} 0"/>
     </link>
     <joint name="${prefix}_knee" type="revolute">

Commit message: will figure out masses and meshes tomrorrow

File: urdf/exov3.urdf.xacro (robot description, xacro)
@@ -17,4 +17,10 @@
     <origin xyz="0 0 1.5" rpy="0 0 0" />
   </joint>
+  <xacro:macro name="point_mass" params="mass">
+    <inertial>
+      <mass value="1.0"/>
+      <inertia ixx="0.01" ixy="0.0" ixz="0.0" iyy="0.01" iyz="0.0" izz="0.01" />
+    </inertial>
+  </xacro:macro>
   <xacro:macro name="motor_cylinder" params="rpy">
     <visual>
@@ -65,4 +71,5 @@
     <link name="${prefix}_calf_link">
       <xacro:common.box width="0.05" depth="0.05" height="0.3" />
+      <xacro:point_mass mass="0.5" />
     </link>
     <joint name="${prefix}_calf" type="fixed">

Commit message: add weighting details + fix frictions

File: urdf/exov3.urdf.xacro (robot description, xacro)
@@ -5,6 +5,14 @@
   <xacro:include filename="materials.xacro" />
   <xacro:property name="steeldensity" value="7850" />
+  <xacro:property name="m_knee" value="5.77" />
+  <xacro:property name="l_calf" value="0.425" />
+  <xacro:property name="lgy_knee" value="0.2633" />
+  <xacro:property name="l_ext" value="0.44" />
+  <xacro:property name="m_ext" value="9.5870" />
+  <xacro:property name="lgy_ext" value="0.1945" />
+  <xacro:property name="lgx_leg" value="0.2095" />
+  <xacro:property name="static_friction" value="10.4160" />
   <xacro:macro name="motor_dynamics">
-      <dynamics damping="0" friction="10.4160" />
+      <dynamics damping="0" friction="${static_friction}" />
   </xacro:macro>
   <link name="world"></link>
@@ -17,8 +25,9 @@
     <origin xyz="0 0 1.5" rpy="0 0 0" />
   </joint>
-  <xacro:macro name="point_mass" params="mass">
+  <xacro:macro name="point_mass" params="mass xyz">
     <inertial>
-      <mass value="1.0"/>
+      <mass value="${mass}"/>
       <inertia ixx="0.01" ixy="0.0" ixz="0.0" iyy="0.01" iyz="0.0" izz="0.01" />
+      <origin xyz="${xyz}" />
     </inertial>
   </xacro:macro>
@@ -46,12 +55,31 @@
     <link name="${prefix}_abduction_link">
       <xacro:motor_cylinder rpy="${pi / 2} 0 0"/>
+      <visual>
+        <geometry>
+          <box size="${lgx_leg} 0.05 0.05" />
+        </geometry>
+        <origin xyz="${multiplier * lgx_leg / 2} 0 0" />
+      </visual>
+      <visual>
+        <geometry>
+          <box size="0.2 0.05 0.05" />
+        </geometry>
+        <origin xyz="${multiplier * lgx_leg} -0.1 0" rpy="0 0 ${pi / 2}"/>
+      </visual>
     </link>
     <link name="${prefix}_hip_link">
       <xacro:motor_cylinder rpy="0 ${pi / 2} 0"/>
+      <visual>
+        <geometry>
+          <box size="0.05 0.05 ${l_ext}" />
+        </geometry>
+        <origin xyz="0 0 ${-1 * l_ext / 2}" />
+      </visual>
+      <xacro:point_mass mass="${m_ext}" xyz="0 0 ${-1 * lgy_ext}"/>
     </link>
     <joint name="${prefix}_hip" type="revolute">
       <parent link="${prefix}_abduction_link" />
       <child link="${prefix}_hip_link" />
-      <origin xyz="${multiplier * 0.2} -0.2 0" rpy="0 0 0" />
+      <origin xyz="${multiplier * lgx_leg} -0.2 0" rpy="0 0 0" />
       <limit lower="${-pi}" upper="${pi}" effort="100" velocity="100" />
       <axis xyz="${multiplier * -1} 0 0" />
@@ -60,21 +88,19 @@
     <link name="${prefix}_knee_link">
       <xacro:motor_cylinder rpy="0 ${pi / 2} 0"/>
+       <visual>
+        <geometry>
+          <box size="0.05 0.05 ${l_calf}" />
+        </geometry>
+        <origin xyz="0 0 ${-1 * l_calf / 2}"/>
+      </visual>
+      <xacro:point_mass mass="${m_knee}" xyz="0 0 ${-1 * lgy_knee}" />
     </link>
     <joint name="${prefix}_knee" type="revolute">
       <parent link="${prefix}_hip_link" />
       <child link="${prefix}_knee_link" />
-      <origin xyz="0 0 -0.5" rpy="0 0 0" />
+      <origin xyz="0 0 ${-1 * l_ext}" rpy="0 0 0" />
       <limit lower="${-pi}" upper="${pi}" effort="100" velocity="100" />
       <axis xyz="${multiplier * -1} 0 0" />
       <xacro:motor_dynamics />
-    </joint>
-    <link name="${prefix}_calf_link">
-      <xacro:common.box width="0.05" depth="0.05" height="0.3" />
-      <xacro:point_mass mass="0.5" />
-    </link>
-    <joint name="${prefix}_calf" type="fixed">
-      <parent link="${prefix}_knee_link" />
-      <child link="${prefix}_calf_link" />
-      <origin xyz="0 0 -0.3" rpy="0 0 0" />
     </joint>
   </xacro:macro>

Commit message: add colors to the urdf

File: urdf/exov3.urdf.xacro (robot description, xacro)
@@ -20,4 +20,7 @@
     <xacro:common.box width="0.3" depth="0.05" height="0.5" density="${steeldensity}" />
   </link>
+  <gazebo reference="base">
+    <material>Gazebo/Black</material>
+  </gazebo>
   <joint name="fix" type="fixed">
     <parent link="world" />
@@ -57,5 +60,5 @@
       <visual>
         <geometry>
-          <box size="${lgx_leg} 0.05 0.05" />
+          <box size="${lgx_leg} 0.04 0.04" />
         </geometry>
         <origin xyz="${multiplier * lgx_leg / 2} 0 0" />
@@ -63,14 +66,17 @@
       <visual>
         <geometry>
-          <box size="0.2 0.05 0.05" />
+          <box size="0.2 0.04 0.04" />
         </geometry>
         <origin xyz="${multiplier * lgx_leg} -0.1 0" rpy="0 0 ${pi / 2}"/>
       </visual>
     </link>
+    <gazebo reference="${prefix}_abduction_link">
+      <material>Gazebo/Red</material>
+    </gazebo>
     <link name="${prefix}_hip_link">
       <xacro:motor_cylinder rpy="0 ${pi / 2} 0"/>
       <visual>
         <geometry>
-          <box size="0.05 0.05 ${l_ext}" />
+          <box size="0.04 0.04 ${l_ext}" />
         </geometry>
         <origin xyz="0 0 ${-1 * l_ext / 2}" />
@@ -78,4 +84,7 @@
       <xacro:point_mass mass="${m_ext}" xyz="0 0 ${-1 * lgy_ext}"/>
     </link>
+    <gazebo reference="${prefix}_hip_link">
+      <material>Gazebo/Black</material>
+    </gazebo>
     <joint name="${prefix}_hip" type="revolute">
       <parent link="${prefix}_abduction_link" />
@@ -90,5 +99,5 @@
        <visual>
         <geometry>
-          <box size="0.05 0.05 ${l_calf}" />
+          <box size="0.04 0.04 ${l_calf}" />
         </geometry>
         <origin xyz="0 0 ${-1 * l_calf / 2}"/>
@@ -96,4 +105,7 @@
       <xacro:point_mass mass="${m_knee}" xyz="0 0 ${-1 * lgy_knee}" />
     </link>
+    <gazebo reference="${prefix}_knee_link">
+      <material>Gazebo/Red</material>
+    </gazebo>
     <joint name="${prefix}_knee" type="revolute">
       <parent link="${prefix}_hip_link" />

Commit message: switch direction of urdf

File: urdf/exov3.urdf.xacro (robot description, xacro)
@@ -132,5 +132,5 @@
     <origin xyz="-0.15 0.05 -0.25" rpy="0 0 0" />
     <limit lower="${-pi / 2}" upper="${pi / 2}" effort="100" velocity="100" />
-    <axis xyz="0 -1 0" />
+    <axis xyz="0 1 0" />
     <xacro:motor_dynamics />
   </joint>
