Commit message: full abstraction of leg

File: urdf/leg/ankle.xacro (robot description, xacro)
@@ -1,5 +1,5 @@
 <?xml version="1.0"?>
 <robot xmlns:xacro="http://www.ros.org/wiki/xacro">
-  <xacro:include filename="common.xacro" />
+  <xacro:include filename="../common.xacro" />
   <xacro:property name="extension_length" value="0.140" />
   <xacro:property name="extension_radius" value="0.013" />

File: urdf/leg/calf.xacro (robot description, xacro)
@@ -1,5 +1,5 @@
 <?xml version="1.0"?>
 <robot xmlns:xacro="http://www.ros.org/wiki/xacro">
-  <xacro:include filename="common.xacro" />
+  <xacro:include filename="../common.xacro" />
   <xacro:property name="plate_length" value="0.100" />
   <xacro:property name="plate_thickness" value="0.087" />

File: urdf/leg/calf_to_ankle.xacro (robot description, xacro)
@@ -1,5 +1,5 @@
 <?xml version="1.0"?>
 <robot xmlns:xacro="http://www.ros.org/wiki/xacro">
-  <xacro:include filename="common.xacro" />
+  <xacro:include filename="../common.xacro" />
   <xacro:include filename="calf.xacro" ns="calf"/>
   <xacro:include filename="ankle.xacro" ns="ankle" />

File: urdf/leg/thigh.xacro (robot description, xacro)
@@ -1,6 +1,6 @@
 <?xml version="1.0"?>
 <robot xmlns:xacro="http://www.ros.org/wiki/xacro">
-  <xacro:include filename="common.xacro" />
-  <xacro:include filename="motor.xacro" ns="motor" />
+  <xacro:include filename="../common.xacro" />
+  <xacro:include filename="../motor.xacro" ns="motor" />
   <xacro:property name="length" value="0.230" />
   <xacro:property name="thickness" value="0.0853" />

File: urdf/v2.urdf.xacro (robot description, xacro)
@@ -5,54 +5,14 @@
   <xacro:include filename="back.xacro" ns="back" />
   <xacro:include filename="motor.xacro" ns="motor" />
-  <xacro:include filename="calf.xacro" ns="calf" />
-  <xacro:include filename="calf_to_ankle.xacro" ns="calf_to_ankle" />
-  <xacro:include filename="thigh.xacro" ns="thigh" />
+  <xacro:include filename="leg/leg.xacro" ns="leg" />
+  <xacro:property name="prefix" value="left" />
   <!-- x = left, y = robot back, z = up -->
   <link name="world"></link>
   <xacro:back.generate_back />
-  <xacro:motor.generate_motor prefix="left_rear" />
+  <xacro:leg.generate_leg prefix="${prefix}" />
   <joint name="left_rear_motor" type="revolute">
     <parent link="back_plate" />
     <child link="left_rear_primary_cylinder" />
     <origin xyz="${back.rear_spacing / 2} ${(back.plate_thickness + motor.thickness) / 2} ${(-1 * back.plate_height / 2) + motor.radius}" rpy="0 0 0" />
-    <limit lower="${-pi / 2}" upper="${pi / 2}" effort="400" velocity="1" />
-    <axis xyz="0 1 0" rpy="0 0 0"/>
-  </joint>
-  <xacro:property name="rear_center_to_edge_length" value="0.130" />
-  <link name="left_rear_limb">
-    <xacro:box_visual_and_collision size="${rear_center_to_edge_length} ${motor.thickness} ${motor.radius * 2}" xyz="0 0 0"/>
-    <xacro:generic_inertia />
-  </link>
-  <joint name="left_rear_limb_to_motor_joint" type="fixed">
-    <parent link="left_rear_secondary_cylinder"/>
-    <child link="left_rear_limb"/>
-    <origin xyz="${rear_center_to_edge_length / 2} 0 0" rpy="0 0 0" />
-  </joint>
-  <xacro:property name="side_plate_length" value="0.260" />
-  <xacro:property name="side_plate_height" value="0.06" />
-  <xacro:property name="side_plate_thickness" value="0.028" />
-  <link name="left_side_plate">
-    <xacro:box_visual_and_collision size="${side_plate_thickness} ${side_plate_length} ${side_plate_height}" xyz="0 0 0" />
-    <xacro:generic_inertia />
-  </link>
-  <joint name="left_side_plate_to_rear_limb" type="fixed">
-    <parent link="left_rear_limb" />
-    <child link="left_side_plate" />
-    <origin xyz="${rear_center_to_edge_length / 2 - side_plate_thickness / 2} ${motor.height / 2 - side_plate_length / 2} 0" />
-  </joint>
-  <xacro:property name="prefix" value="left" />
-  <xacro:thigh.generate_thigh prefix="${prefix}" />
-  <joint name="left_hip_motor" type="revolute">
-    <parent link="left_side_plate" />
-    <child link="left_hip_primary_cylinder" />
-    <origin xyz="${-1 * motor.thickness / 2} ${-1 * side_plate_length / 2} 0" rpy="0 ${pi/2} ${pi / 2}" />
-    <limit lower="${-pi / 2}" upper="${pi / 2}" effort="400" velocity="1" />
-    <axis xyz="0 1 0" rpy="0 0 0"/>
-  </joint>
-  <xacro:calf_to_ankle.generate_calf_to_ankle prefix="${prefix}" />
-  <joint name="left_knee_to_calf" type="revolute">
-    <parent link="left_knee_secondary_cylinder" />
-    <child link="left_calf_plate" />
-    <origin xyz="${calf.plate_length / 2} ${(motor.thickness + calf.plate_width) / 2} 0" rpy="0 0 0" />
     <limit lower="${-pi / 2}" upper="${pi / 2}" effort="400" velocity="1" />
     <axis xyz="0 1 0" rpy="0 0 0"/>
