Commit message: encoder gaming

File: urdf/leg/leg.xacro (robot description, xacro)
@@ -13,6 +13,7 @@
       <child link="${prefix}_hip_primary_cylinder" />
       <origin xyz="${-1 * motor.thickness / 2} ${-1 * rear_limb.side_plate_length / 2} 0" rpy="0 ${pi/2} ${pi / 2}" />
-      <limit lower="${-pi / 2}" upper="${pi / 2}" effort="400" velocity="1" />
+      <limit lower="${-pi / 2}" upper="${pi / 2}" effort="400" velocity="100" />
       <axis xyz="0 1 0" rpy="0 0 0"/>
+      <dynamics damping="0.3" />
     </joint>
     <xacro:calf_to_ankle.generate_calf_to_ankle prefix="${prefix}" />
@@ -21,6 +22,7 @@
       <child link="${prefix}_calf_plate" />
       <origin xyz="${calf.plate_length / 2} ${(motor.thickness + calf.plate_width) / 2} 0" rpy="0 0 0" />
-      <limit lower="${-pi / 2}" upper="${pi / 2}" effort="400" velocity="1" />
+      <limit lower="${-pi / 2}" upper="${pi / 2}" effort="400" velocity="100" />
       <axis xyz="0 1 0" rpy="0 0 0"/>
+      <dynamics damping="0.3" />
     </joint>
   </xacro:macro>

File: urdf/v2.urdf.xacro (robot description, xacro)
@@ -11,9 +11,10 @@
   <xacro:back.generate_back />
   <xacro:leg.generate_leg prefix="${prefix}" />
-  <joint name="left_rear_motor" type="revolute">
+  <joint name="left_rear_motor" type="fixed">
     <parent link="back_plate" />
     <child link="left_rear_primary_cylinder" />
     <origin xyz="${back.rear_spacing / 2} ${(back.plate_thickness + motor.thickness) / 2} ${(-1 * back.plate_height / 2) + motor.radius}" rpy="0 0 0" />
-    <limit lower="${-pi / 2}" upper="${pi / 2}" effort="400" velocity="1" />
+    <limit lower="${-pi / 2}" upper="${pi / 2}" effort="400" velocity="100" />
+    <dynamics damping="0.3" />
     <axis xyz="0 1 0" rpy="0 0 0"/>
   </joint>

Commit message: add friction

File: urdf/leg/leg.xacro (robot description, xacro)
@@ -15,5 +15,5 @@
       <limit lower="${-pi / 2}" upper="${pi / 2}" effort="400" velocity="100" />
       <axis xyz="0 1 0" rpy="0 0 0"/>
-      <dynamics damping="0.3" />
+      <dynamics damping="0.1" friction="0.1" />
     </joint>
     <xacro:calf_to_ankle.generate_calf_to_ankle prefix="${prefix}" />
@@ -24,5 +24,5 @@
       <limit lower="${-pi / 2}" upper="${pi / 2}" effort="400" velocity="100" />
       <axis xyz="0 1 0" rpy="0 0 0"/>
-      <dynamics damping="0.3" />
+      <dynamics damping="0.1" friction="0.1"/>
     </joint>
   </xacro:macro>
